File: _autosave-MX_IMU.kicad_sch (KiCad schematic)
At the start: 31 parts, among them U1 STM32F405RGT6, U3 ld39150dt33-r, Y1 16MHz

Commit message: save
Parts:
- D1, D2, D3: footprint mylib:CHIPLED_0603_NOOUTLINE -> LED_SMD:LED_0603_1608Metric
Changed lines of the file:
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@@
 			)
 		)
-		(property "Footprint" "mylib:CHIPLED_0603_NOOUTLINE"
+		(property "Footprint" "LED_SMD:LED_0603_1608Metric"
 			(at 232.41 33.02 0)
 			(effects
@@
 			)
 		)
-		(property "Footprint" "mylib:CHIPLED_0603_NOOUTLINE"
+		(property "Footprint" "LED_SMD:LED_0603_1608Metric"
 			(at 254 87.63 0)
 			(effects
@@
 			)
 		)
-		(property "Footprint" "mylib:CHIPLED_0603_NOOUTLINE"
+		(property "Footprint" "LED_SMD:LED_0603_1608Metric"
 			(at 266.7 87.63 0)
 			(effects
