File: _autosave-MX_IMU.kicad_sch (KiCad schematic)
At the start: 24 parts, among them U1 STM32F405RGT6, Y1 16MHz

Commit message: update
Parts:
- renumbered C28 to C13
Other:
- note removed: ""ON" LED"
- note removed: "RGB LED ( NEOPIXEL )"
- moved on the sheet: C13, D1
