File: MX_IMU.kicad_sch (KiCad schematic)
At the start: 31 parts, among them U1 STM32F405RGT6, U3 ld39150dt33-r, Y1 16MHz

Commit message: update pcb
Parts:
- removed C13: 1u, Capacitor_SMD:C_0603_1608Metric, symbol Device:C
- removed C14: 2u2, Capacitor_SMD:C_0603_1608Metric, symbol Device:C_Small
- removed D1: GREEN, mylib:CHIPLED_0603_NOOUTLINE, symbol Device:LED
- removed R6: 10k, Resistor_SMD:R_0402_1005Metric, symbol Device:R_Small
- removed U3: ld39150dt33-r, common:to-252-2_dpak-2-leg, symbol common:ld39150dt33-r
- D1: renamed from D2; footprint mylib:CHIPLED_0603_NOOUTLINE -> LED_SMD:LED_0603_1608Metric
- D2: renamed from D3; footprint mylib:CHIPLED_0603_NOOUTLINE -> LED_SMD:LED_0603_1608Metric
- renumbered R3 to R1, R4 to R2, R5 to R3, R7 to R4, R8 to R5
Connections:
- net USART4_RX renamed USART3_RX
- net USART4_TX renamed USART3_TX
Other:
- added sheet PowerSupply (PowerSupply.kicad_sch)
