File: MX_IMU.kicad_sch (KiCad schematic)
At the start: 4 parts

Commit message: update
Other:
- sheet PowerAndUSB renamed (lib_symbols 	(symbol "SSSS213000:SSSS213000" 		(exclude_from_sim no) 		(in_bom yes) 		(on_board yes) 		(property "Reference" "D" 			(at 19.05 7.62 0) 			(effects 				(font (size 1.27 1.27)) 				(justify left top) 			) 		) 		(property "Value" "SSSS213000" 			(at 19.05 5.08 0) 			(effects 				(font (size 1.27 1.27)) 				(justify left top) 			) 		) 		(property "Footprint" "SSSS213000" 			(at 19.05 -94.92 0) 			(effects 				(font (size 1.27 1.27)) 				(justify left top) 				(hide yes) 			) 		) 		(property "Datasheet" "https://www.alps.com/prod/info/E/HTML/Switch/Slide/SSSS2/SSSS213000.html" 			(at 19.05 -194.92 0) 			(effects 				(font (size 1.27 1.27)) 				(justify left top) 				(hide yes) 			) 		) 		(property "Description" "Slide Switches 1-pole 2-positions" 			(at 0 0 0) 			(effects 				(font (size 1.27 1.27)) 				(hide yes) 			) 		) 		(property "Height" "5" 			(at 19.05 -394.92 0) 			(effects 				(font (size 1.27 1.27)) 				(justify left top) 				(hide yes) 			) 		) 		(property "Avnet Part Number" "" 			(at 19.05 -494.92 0) 			(effects 				(font (size 1.27 1.27)) 				(justify left top) 				(hide yes) 			) 		) 		(property "Avnet Price/Stock" "" 			(at 19.05 -594.92 0) 			(effects 				(font (size 1.27 1.27)) 				(justify left top) 				(hide yes) 			) 		) 		(property "Manufacturer_Name" "ALPS Electric" 			(at 19.05 -694.92 0) 			(effects 				(font (size 1.27 1.27)) 				(justify left top) 				(hide yes) 			) 		) 		(property "Manufacturer_Part_Number" "SSSS213000" 			(at 19.05 -794.92 0) 			(effects 				(font (size 1.27 1.27)) 				(justify left top) 				(hide yes) 			) 		) 		(symbol "SSSS213000_1_1" 			(rectangle 				(start 5.08 2.54) 				(end 17.78 -5.08) 				(stroke (width 0.254) (type default)) 				(fill (type background)) 			) 			(pin passive line 				(at 0 0 0) 				(length 5.08) 				(name "C" 					(effects 						(font (size 1.27 1.27)) 					) 				) 				(number "2" 					(effects 						(font (size 1.27 1.27)) 					) 				) 			) 			(pin no_connect line 				(at 22.86 0 180) 				(length 5.08) 				(name "NC" 					(effects 						(font (size 1.27 1.27)) 					) 				) 				(number "3" 					(effects 						(font (size 1.27 1.27)) 					) 				) 			) 			(pin passive line 				(at 22.86 -2.54 180) 				(length 5.08) 				(name "NO" 					(effects 						(font (size 1.27 1.27)) 					) 				) 				(number "1" 					(effects 						(font (size 1.27 1.27)) 					) 				) 			) 		) 		(embedded_fonts no) 	) ) (symbol 	(lib_id "SSSS213000:SSSS213000") 	(at 168.91 143.51 180) 	(unit 1) 	(exclude_from_sim no) 	(in_bom yes) 	(on_board yes) 	(dnp no) 	(uuid "1cfbf113-b454-4c9b-a589-10a73b0e294d") 	(property "Reference" "SW1" 		(at 157.48 135.636 0) 		(effects 			(font (size 1.27 1.27)) 			(justify left) 		) 	) 	(property "Value" "SSSS213000" 		(at 157.4801 156.21 90) 		(effects 			(font (size 1.27 1.27)) 			(justify left) 			(hide yes) 		) 	) 	(property "Footprint" "mylib:SSSS213000" 		(at 149.86 48.59 0) 		(effects 			(font (size 1.27 1.27)) 			(justify left top) 			(hide yes) 		) 	) 	(property "Datasheet" "https://www.alps.com/prod/info/E/HTML/Switch/Slide/SSSS2/SSSS213000.html" 		(at 149.86 -51.41 0) 		(effects 			(font (size 1.27 1.27)) 			(justify left top) 			(hide yes) 		) 	) 	(property "Description" "Slide Switches 1-pole 2-positions" 		(at 168.91 143.51 0) 		(effects 			(font (size 1.27 1.27)) 			(hide yes) 		) 	) 	(property "Height" "5" 		(at 149.86 -251.41 0) 		(effects 			(font (size 1.27 1.27)) 			(justify left top) 			(hide yes) 		) 	) 	(property "Avnet Part Number" "" 		(at 149.86 -351.41 0) 		(effects 			(font (size 1.27 1.27)) 			(justify left top) 			(hide yes) 		) 	) 	(property "Avnet Price/Stock" "" 		(at 149.86 -451.41 0) 		(effects 			(font (size 1.27 1.27)) 			(justify left top) 			(hide yes) 		) 	) 	(property "Manufacturer_Name" "ALPS Electric" 		(at 149.86 -551.41 0) 		(effects 			(font (size 1.27 1.27)) 			(justify left top) 			(hide yes) 		) 	) 	(property "Manufacturer_Part_Number" "SSSS213000" 		(at 149.86 -651.41 0) 		(effects 			(font (size 1.27 1.27)) 			(justify left top) 			(hide yes) 		) 	) 	(pin "3" 		(uuid "baaf3ec1-1186-40a8-835a-1680c7c84360") 	) 	(pin "1" 		(uuid "827880ac-dff7-40fc-8467-e6db01118f5e") 	) 	(pin "2" 		(uuid "fd02f8df-5769-4a7f-80bc-813f43238c94") 	) 	(instances 		(project "MX_IMU" 			(path "" 				(reference "SW1") 				(unit 1) 			) 		) 	) )
Changed lines of the file:
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@@
 			(color 0 0 0 0.0000)
-		)
-		(property "Sheetname" "PowerAndUSB"
-			(at 93.98 87.5534 0)
-			(effects
-				(font
-					(size 2.54 2.54)
-					(thickness 0.508)
-					(bold yes)
-				)
-				(justify left bottom)
-			)
 		)
 		(property "Sheetfile" "PowerSupply.kicad_sch"
