File: MX_IMU.kicad_sch (KiCad schematic)
At the start: 24 parts, among them U1 STM32F405RGT6, Y1 16MHz

Commit message: update
Parts:
- removed C1: 4u7, Capacitor_SMD:C_0603_1608Metric, symbol Device:C_Small
- removed C10: 10n, Capacitor_SMD:C_0402_1005Metric, symbol Device:C_Small
- removed C11, C12: 12p, Capacitor_SMD:C_0402_1005Metric, symbol Device:C_Small
- removed C2, C3: 2u2, Capacitor_SMD:C_0603_1608Metric, symbol Device:C_Small
- removed C28: 100nf, Capacitor_SMD:C_0603_1608Metric, symbol Device:C_Small
- removed C4, C5, C6, C7, C8: 100n, Capacitor_SMD:C_0402_1005Metric, symbol Device:C_Small
- removed C9: 1u, Capacitor_SMD:C_0402_1005Metric, symbol Device:C_Small
- removed D1: WS2812, LED_SMD:LED_WS2812_PLCC6_5.0x5.0mm_P1.6mm, symbol LED:WS2812
- removed FB1: 600 @ 600 MHz, Inductor_SMD:L_0805_2012Metric, symbol Device:FerriteBead_Small
- removed R1: 47, Resistor_SMD:R_0402_1005Metric, symbol Device:R_Small
- removed R2: 10k, Resistor_SMD:R_0603_1608Metric, symbol Device:R
- removed R3: 10k, Resistor_SMD:R_0402_1005Metric, symbol Device:R_Small
- removed U1: STM32F405RGT6, Package_QFP:LQFP-64_10x10mm_P0.5mm, symbol MCU_ST_STM32F4:STM32F405RGTx
- removed Y1: 16MHz, Crystal:Crystal_SMD_3225-4Pin_3.2x2.5mm, symbol Device:Crystal_GND24_Small
Connections:
- no-connect marks 32 -> 0
Other:
- sheet PowerSupply renamed PowerAndUSB
- added sheet MCU (MCU.kicad_sch)
- added sheet sensor (sensor.kicad_sch)
- sheet Connectors ports: added none; removed CAN2_RX, CAN2_TX
- note added: "Mounting holes"
- note removed: ""ON" LED"
- note removed: "BOOT0 Switch"
- note removed: "Decoupling"
- note removed: "HSE"
- note removed: "Mounting Holes"
- note removed: "RGB LED ( NEOPIXEL )"
- note removed: "STM32 MCU"
- note removed: "Status LEDs"
- moved on the sheet: H1, H2, H3, H4

Commit message: update
Other:
- sheet sensor renamed Peripherals
- sheet Peripherals: file sensor.kicad_sch -> Periph.kicad_sch
Changed lines of the file:
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@@
 			(color 0 0 0 0.0000)
 		)
-		(property "Sheetname" "sensor"
+		(property "Sheetname" "Peripherals"
 			(at 93.98 121.8434 0)
 			(effects
@@
 			)
 		)
-		(property "Sheetfile" "sensor.kicad_sch"
+		(property "Sheetfile" "Periph.kicad_sch"
 			(at 93.98 149.1746 0)
 			(effects

Commit message: compact  IMU module for integration
Parts:
- H1, H2, H3, H4: footprint MountingHole:MountingHole_3.2mm_M3_Pad_Via -> MountingHole:MountingHole_2.2mm_M2_DIN965_Pad
