File: Connectors.kicad_sch (KiCad schematic)
At the start: 21 parts, among them J1 353630460, J3 2171750001, J4 353630660, J5 353630660, U4 TJA1051T/3, U5 ICM-42688-P

Commit message: update pcb
Parts:
- removed J3: 2171750001, common:molex_2171750001_usb_c_6p, symbol common:molex_2171750001_usb_c_6p
- removed R1, R2: 5k1, Resistor_SMD:R_0603_1608Metric, symbol Device:R

Commit message: save
Parts:
- renumbered C400 to C15, C2 to C16, C31 to C17, C1 to C18, C4 to C19, C10 to C20, J5 to J1, J4 to J2, J1 to J3, R401 to R10, R400 to R11, R19 to R12, R20 to R13, R406 to R14, R407 to R15, R403 to R9

Commit message: update pcb
Parts:
- removed J3: 353630460, mylib:CON_353630460, symbol 353630460:353630460
- renumbered C15 to C13, C16 to C14, C17 to C15, C18 to C16, C19 to C17, C20 to C18, R13 to R10, R14 to R11, R15 to R12, R9 to R6, R10 to R7, R11 to R8, R12 to R9, U4 to U2, U5 to U3
Connections:
- net +5V: no longer J2.1
- no-connect marks 5 -> 6
Other:
- note removed: "GPS_UART"

Commit message: update
Parts:
- removed C16: 0.1u, Capacitor_SMD:C_0402_1005Metric, symbol Device:C_Small
- removed C17: 2u2, Capacitor_SMD:C_0603_1608Metric, symbol Device:C_Small
- removed C18: 10n, Capacitor_SMD:C_0402_1005Metric, symbol Device:C_Small
- removed J1: 353630660, mylib:CON_353630660, symbol 353630660:353630660
- removed U3: ICM-42688-P, mylib:PQFN50P300X250X97-14N, symbol ICM-42688-P:ICM-42688-P
- added J7: SWD, Connector_PinHeader_2.54mm:PinHeader_1x06_P2.54mm_Vertical, symbol Connector_Generic:Conn_01x06
- renumbered C14 to C27, C15 to C28, C13 to C29, J2 to J4, R11 to R12, R12 to R13, R9 to R14, R10 to R15, R7 to R16, R8 to R17, R6 to R18, U2 to U9
Connections:
- net +3.3V: now also J7.6 (Pin_6)
- net GND: now also J7.5 (Pin_5)
- net SWO: now also J7.1 (Pin_1)
- net at R17.2: now also J7.3 (Pin_3)
- net at R16.2: now also J7.2 (Pin_2)
- net at R18.2: now also J7.4 (Pin_4)
- no-connect marks 6 -> 1
Other:
- note removed: "IMU-ICM42688P"
- moved on the sheet: C29, R16, R17, R18

Commit message: update library
Parts:
- C28: renamed from C27; value 100n -> C_Small
- C29: renamed from C28; value 4n7 -> C
- C30: renamed from C29; value 100n -> C_Small
- J4: footprint mylib:CON_353630660 -> 353630660:CON_353630660
- J5: renamed from J7; value SWD -> Conn_01x06
- R15: renamed from R12; value 22 -> R_Small
- R16: renamed from R13; value 22 -> R_Small
- R17: renamed from R14; value 60R -> R
- R18: renamed from R15; value 60R -> R
- R19: renamed from R16; value 22 -> R_Small
- R20: renamed from R17; value 22 -> R_Small
- R21: renamed from R18; value 22 -> R_Small
- renumbered U9 to U10
Changed lines of the file:
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@@
 		(on_board yes)
 		(dnp no)
-		(property "Reference" "#PWR067"
+		(property "Reference" "#PWR073"
 			(at 120.65 80.01 0)
 			(effects
@@
 			(project "MX_IMU"
 				(path "/8ed38441-7d4e-4e89-870f-07e11c6dce38/3e6b1080-2480-49a7-8bae-2dbfae5f98f5"
-					(reference "#PWR067")
+					(reference "#PWR073")
 					(unit 1)
 				)
@@
 		(on_board yes)
 		(dnp no)
-		(property "Reference" "R12"
+		(property "Reference" "R15"
 			(at 118.11 59.69 90)
 			(effects
@@
 			)
 		)
-		(property "Value" "22"
+		(property "Value" "R_Small"
 			(at 118.11 62.23 90)
 			(effects
@@
 			(project "MX_IMU"
 				(path "/8ed38441-7d4e-4e89-870f-07e11c6dce38/3e6b1080-2480-49a7-8bae-2dbfae5f98f5"
-					(reference "R12")
+					(reference "R15")
 					(unit 1)
 				)
@@
 		(on_board yes)
 		(dnp no)
-		(property "Reference" "R13"
+		(property "Reference" "R16"
 			(at 118.11 67.31 90)
 			(effects
@@
 			)
 		)
-		(property "Value" "22"
+		(property "Value" "R_Small"
 			(at 118.11 64.77 90)
 			(effects
@@
 			(project "MX_IMU"
 				(path "/8ed38441-7d4e-4e89-870f-07e11c6dce38/3e6b1080-2480-49a7-8bae-2dbfae5f98f5"
-					(reference "R13")
+					(reference "R16")
 					(unit 1)
 				)
@@
 		(on_board yes)
 		(dnp no)
-		(property "Reference" "R17"
+		(property "Reference" "R20"
 			(at 68.58 144.78 90)
 			(effects
@@
 			)
 		)
-		(property "Value" "22"
+		(property "Value" "R_Small"
 			(at 68.58 142.24 90)
 			(effects
@@
 			(project "MX_IMU"
 				(path "/8ed38441-7d4e-4e89-870f-07e11c6dce38/3e6b1080-2480-49a7-8bae-2dbfae5f98f5"
-					(reference "R17")
+					(reference "R20")
 					(unit 1)
 				)
@@
 		(on_board yes)
 		(dnp no)
-		(property "Reference" "R16"
+		(property "Reference" "R19"
 			(at 68.58 138.176 90)
 			(effects
@@
 			)
 		)
-		(property "Value" "22"
+		(property "Value" "R_Small"
 			(at 68.58 139.7 90)
 			(effects
@@
 			(project "MX_IMU"
 				(path "/8ed38441-7d4e-4e89-870f-07e11c6dce38/3e6b1080-2480-49a7-8bae-2dbfae5f98f5"
-					(reference "R16")
+					(reference "R19")
 					(unit 1)
 				)
@@
 		(on_board yes)
 		(dnp no)
-		(property "Reference" "R18"
+		(property "Reference" "R21"
 			(at 53.34 157.48 90)
 			(effects
@@
 			)
 		)
-		(property "Value" "22"
+		(property "Value" "R_Small"
 			(at 54.61 154.94 90)
 			(effects
@@
 			(project "MX_IMU"
 				(path "/8ed38441-7d4e-4e89-870f-07e11c6dce38/3e6b1080-2480-49a7-8bae-2dbfae5f98f5"
-					(reference "R18")
+					(reference "R21")
 					(unit 1)
 				)
@@
 		(on_board yes)
 		(dnp no)
-		(property "Reference" "C29"
+		(property "Reference" "C30"
 			(at 48.4632 151.0284 0)
 			(effects
@@
 			)
 		)
-		(property "Value" "100n"
+		(property "Value" "C_Small"
 			(at 48.4632 148.717 0)
 			(effects
@@
 			(project "MX_IMU"
 				(path "/8ed38441-7d4e-4e89-870f-07e11c6dce38/3e6b1080-2480-49a7-8bae-2dbfae5f98f5"
-					(reference "C29")
+					(reference "C30")
 					(unit 1)
 				)
@@
 		(on_board yes)
 		(dnp no)
-		(property "Reference" "#PWR072"
+		(property "Reference" "#PWR078"
 			(at 67.31 146.05 0)
 			(effects
@@
 			(project "MX_IMU"
 				(path "/8ed38441-7d4e-4e89-870f-07e11c6dce38/3e6b1080-2480-49a7-8bae-2dbfae5f98f5"
-					(reference "#PWR072")
+					(reference "#PWR078")
 					(unit 1)
 				)
@@
 		(on_board yes)
 		(dnp no)
-		(property "Reference" "#PWR071"
+		(property "Reference" "#PWR077"
 			(at 66.04 147.32 0)
 			(effects
@@
 			(project "MX_IMU"
 				(path "/8ed38441-7d4e-4e89-870f-07e11c6dce38/3e6b1080-2480-49a7-8bae-2dbfae5f98f5"
-					(reference "#PWR071")
+					(reference "#PWR077")
 					(unit 1)
 				)
@@
 		(on_board yes)
 		(dnp no)
-		(property "Reference" "#PWR070"
+		(property "Reference" "#PWR076"
 			(at 50.8 140.97 0)
 			(effects
@@
 			(project "MX_IMU"
 				(path "/8ed38441-7d4e-4e89-870f-07e11c6dce38/3e6b1080-2480-49a7-8bae-2dbfae5f98f5"
-					(reference "#PWR070")
+					(reference "#PWR076")
 					(unit 1)
 				)
@@
 		(dnp no)
 		(fields_autoplaced yes)
-		(property "Reference" "#PWR068"
+		(property "Reference" "#PWR074"
 			(at 62.23 83.82 0)
 			(effects
@@
 			(project "MX_IMU"
 				(path "/8ed38441-7d4e-4e89-870f-07e11c6dce38/3e6b1080-2480-49a7-8bae-2dbfae5f98f5"
-					(reference "#PWR068")
+					(reference "#PWR074")
 					(unit 1)
 				)
@@
 		(dnp no)
 		(fields_autoplaced yes)
-		(property "Reference" "#PWR064"
+		(property "Reference" "#PWR071"
 			(at 80.01 57.15 0)
 			(effects
@@
 			(project "MX_IMU"
 				(path "/8ed38441-7d4e-4e89-870f-07e11c6dce38/3e6b1080-2480-49a7-8bae-2dbfae5f98f5"
-					(reference "#PWR064")
+					(reference "#PWR071")
 					(unit 1)
 				)
@@
 		(on_board yes)
 		(dnp no)
-		(property "Reference" "#PWR066"
+		(property "Reference" "#PWR072"
 			(at 44.45 68.58 0)
 			(effects
@@
 			(project "MX_IMU"
 				(path "/8ed38441-7d4e-4e89-870f-07e11c6dce38/3e6b1080-2480-49a7-8bae-2dbfae5f98f5"
-					(reference "#PWR066")
+					(reference "#PWR072")
 					(unit 1)
 				)
@@
 		(dnp no)
 		(fields_autoplaced yes)
-		(property "Reference" "J7"
+		(property "Reference" "J5"
 			(at 81.28 142.2399 0)
 			(effects
@@
 			)
 		)
-		(property "Value" "SWD"
+		(property "Value" "Conn_01x06"
 			(at 81.28 144.7799 0)
 			(effects
@@
 			(project "MX_IMU"
 				(path "/8ed38441-7d4e-4e89-870f-07e11c6dce38/3e6b1080-2480-49a7-8bae-2dbfae5f98f5"
-					(reference "J7")
+					(reference "J5")
 					(unit 1)
 				)
@@
 		(on_board yes)
 		(dnp no)
-		(property "Reference" "C28"
+		(property "Reference" "C29"
 			(at 92.71 83.82 0)
 			(effects
@@
 			)
 		)
-		(property "Value" "4n7"
+		(property "Value" "C"
 			(at 92.71 86.36 0)
 			(effects
@@
 			(project "MX_IMU"
 				(path "/8ed38441-7d4e-4e89-870f-07e11c6dce38/3e6b1080-2480-49a7-8bae-2dbfae5f98f5"
-					(reference "C28")
+					(reference "C29")
 					(unit 1)
 				)
@@
 		(dnp no)
 		(fields_autoplaced yes)
-		(property "Reference" "#PWR063"
+		(property "Reference" "#PWR070"
 			(at 77.47 44.45 0)
 			(effects
@@
 			(project ""
 				(path "/8ed38441-7d4e-4e89-870f-07e11c6dce38/3e6b1080-2480-49a7-8bae-2dbfae5f98f5"
-					(reference "#PWR063")
+					(reference "#PWR070")
 					(unit 1)
 				)
@@
 		(on_board yes)
 		(dnp no)
-		(property "Reference" "R14"
+		(property "Reference" "R17"
 			(at 86.614 73.66 0)
 			(effects
@@
 			)
 		)
-		(property "Value" "60R"
+		(property "Value" "R"
 			(at 86.614 76.2 0)
 			(effects
@@
 			(project "MX_IMU"
 				(path "/8ed38441-7d4e-4e89-870f-07e11c6dce38/3e6b1080-2480-49a7-8bae-2dbfae5f98f5"
-					(reference "R14")
+					(reference "R17")
 					(unit 1)
 				)
@@
 		(dnp no)
 		(fields_autoplaced yes)
-		(property "Reference" "#PWR069"
+		(property "Reference" "#PWR075"
 			(at 90.17 96.52 0)
 			(effects
@@
 			(project "MX_IMU"
 				(path "/8ed38441-7d4e-4e89-870f-07e11c6dce38/3e6b1080-2480-49a7-8bae-2dbfae5f98f5"
-					(reference "#PWR069")
+					(reference "#PWR075")
 					(unit 1)
 				)
@@
 		(on_board yes)
 		(dnp no)
-		(property "Reference" "U9"
+		(property "Reference" "U10"
 			(at 73.152 55.118 0)
 			(effects
@@
 			(project "MX_IMU"
 				(path "/8ed38441-7d4e-4e89-870f-07e11c6dce38/3e6b1080-2480-49a7-8bae-2dbfae5f98f5"
-					(reference "U9")
+					(reference "U10")
 					(unit 1)
 				)
@@
 		(on_board yes)
 		(dnp no)
-		(property "Reference" "R15"
+		(property "Reference" "R18"
 			(at 96.774 73.66 0)
 			(effects
@@
 			)
 		)
-		(property "Value" "60R"
+		(property "Value" "R"
 			(at 96.774 76.2 0)
 			(effects
@@
 			(project "MX_IMU"
 				(path "/8ed38441-7d4e-4e89-870f-07e11c6dce38/3e6b1080-2480-49a7-8bae-2dbfae5f98f5"
-					(reference "R15")
+					(reference "R18")
 					(unit 1)
 				)
@@
 		(on_board yes)
 		(dnp no)
-		(property "Reference" "C27"
+		(property "Reference" "C28"
 			(at 82.55 43.18 0)
 			(effects
@@
 			)
 		)
-		(property "Value" "100n"
+		(property "Value" "C_Small"
 			(at 82.55 45.72 0)
 			(effects
@@
 			(project "MX_IMU"
 				(path "/8ed38441-7d4e-4e89-870f-07e11c6dce38/3e6b1080-2480-49a7-8bae-2dbfae5f98f5"
-					(reference "C27")
+					(reference "C28")
 					(unit 1)
 				)
@@
 			)
 		)
-		(property "Footprint" "mylib:CON_353630660"
+		(property "Footprint" "353630660:CON_353630660"
 			(at 120.65 59.69 0)
 			(effects

Commit message: clean files
Parts:
- removed J4: 353630660, 353630660:CON_353630660, symbol 353630660:353630660
- added J4: Conn_01x06, Connector_PinHeader_2.54mm:PinHeader_1x06_P2.54mm_Vertical, symbol Connector_Generic:Conn_01x06
Connections:
- net CAN2+: now also J4.4 (Pin_4)
- net CAN2-: now also J4.5 (Pin_5)
- net GND: now also J4.6 (Pin_6)
- net at R15.1: now also J4.2 (Pin_2)
- net at R16.1: now also J4.3 (Pin_3)
Changed lines of the file:
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@@
+	)
+	(symbol
+		(lib_id "Connector_Generic:Conn_01x06")
+		(at 125.73 64.77 0)
+		(unit 1)
+		(exclude_from_sim no)
+		(in_bom yes)
+		(on_board yes)
+		(dnp no)
+		(fields_autoplaced yes)
+		(property "Reference" "J4"
+			(at 128.27 64.7699 0)
+			(effects
+				(font
+					(size 1.27 1.27)
+				)
+				(justify left)
+			)
+		)
+		(property "Value" "Conn_01x06"
+			(at 128.27 67.3099 0)
+			(effects
+				(font
+					(size 1.27 1.27)
+				)
+				(justify left)
+			)
+		)
+		(property "Footprint" "Connector_PinHeader_2.54mm:PinHeader_1x06_P2.54mm_Vertical"
+			(at 125.73 64.77 0)
+			(effects
+				(font
+					(size 1.27 1.27)
+				)
+				(hide yes)
+			)
+		)
+		(property "Datasheet" "~"
+			(at 125.73 64.77 0)
+			(effects
+				(font
+					(size 1.27 1.27)
+				)
+				(hide yes)
+			)
+		)
+		(property "Description" ""
+			(at 125.73 64.77 0)
+			(effects
+				(font
+					(size 1.27 1.27)
+				)
+			)
+		)
+		(pin "1"
+		)
+		(pin "2"
+		)
+		(pin "3"
+		)
+		(pin "4"
+		)
+		(pin "5"
+		)
+		(pin "6"
+		)
+		(instances
+			(project "MX_IMU"
+				(path "/8ed38441-7d4e-4e89-870f-07e11c6dce38/3e6b1080-2480-49a7-8bae-2dbfae5f98f5"
+					(reference "J4")
+					(unit 1)
+				)
+			)
+		)
 	)
 	(symbol
@@
 					(unit 1)
 				)
-			)
-		)
-	)
-	(symbol
-		(lib_id "353630660:353630660")
-		(at 120.65 59.69 0)
-		(unit 1)
-		(exclude_from_sim no)
-		(in_bom yes)
-		(on_board yes)
-		(dnp no)
-		(fields_autoplaced yes)
-		(property "Reference" "J4"
-			(at 135.001 64.7699 0)
-			(effects
-				(font
-					(size 1.27 1.27)
-				)
-				(justify left)
-			)
-		)
-		(property "Value" "353630660"
-			(at 135.001 67.3099 0)
-			(effects
-				(font
-					(size 1.27 1.27)
-				)
-				(justify left)
-				(hide yes)
-			)
-		)
-		(property "Footprint" "353630660:CON_353630660"
-			(at 120.65 59.69 0)
-			(effects
-				(font
-					(size 1.27 1.27)
-				)
-				(justify bottom)
-				(hide yes)
-			)
-		)
-		(property "Datasheet" ""
-			(at 120.65 59.69 0)
-			(effects
-				(font
-					(size 1.27 1.27)
-				)
-				(hide yes)
-			)
-		)
-		(property "Description" ""
-			(at 120.65 59.69 0)
-			(effects
-				(font
-					(size 1.27 1.27)
-				)
-				(hide yes)
-			)
-		)
-		(property "MFR_NAME" "Molex Connector Corporation"
-			(at 120.65 59.69 0)
-			(effects
-				(font
-					(size 1.27 1.27)
-				)
-				(justify bottom)
-				(hide yes)
-			)
-		)
-		(property "MANUFACTURER_PART_NUMBER" "353630660"
-			(at 120.65 59.69 0)
-			(effects
-				(font
-					(size 1.27 1.27)
-				)
-				(justify bottom)
-				(hide yes)
-			)
-		)
-		(pin "1"
-		)
-		(pin "2"
-		)
-		(pin "4"
-		)
-		(pin "6"
-		)
-		(pin "5"
-		)
-		(pin "3"
-		)
-		(instances
-			(project "MX_IMU"
-				(path "/8ed38441-7d4e-4e89-870f-07e11c6dce38/3e6b1080-2480-49a7-8bae-2dbfae5f98f5"
-					(reference "J4")
-					(unit 1)
-				)

Commit message: update
Parts:
- renumbered C30 to C28, C28 to C29, C29 to C30, J5 to J4, J4 to J5, R21 to R15, R19 to R16, R20 to R17, R17 to R18, R18 to R19, R15 to R20, R16 to R21
Changed lines of the file:
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@@
 		(on_board yes)
 		(dnp no)
-		(property "Reference" "#PWR073"
+		(property "Reference" "#PWR078"
 			(at 120.65 80.01 0)
 			(effects
@@
 			(project "MX_IMU"
 				(path "/8ed38441-7d4e-4e89-870f-07e11c6dce38/3e6b1080-2480-49a7-8bae-2dbfae5f98f5"
-					(reference "#PWR073")
+					(reference "#PWR078")
 					(unit 1)
 				)
@@
 		(on_board yes)
 		(dnp no)
-		(property "Reference" "R15"
+		(property "Reference" "R20"
 			(at 118.11 59.69 90)
 			(effects
@@
 			(project "MX_IMU"
 				(path "/8ed38441-7d4e-4e89-870f-07e11c6dce38/3e6b1080-2480-49a7-8bae-2dbfae5f98f5"
-					(reference "R15")
+					(reference "R20")
 					(unit 1)
 				)
@@
 		(on_board yes)
 		(dnp no)
-		(property "Reference" "R16"
+		(property "Reference" "R21"
 			(at 118.11 67.31 90)
 			(effects
@@
 			(project "MX_IMU"
 				(path "/8ed38441-7d4e-4e89-870f-07e11c6dce38/3e6b1080-2480-49a7-8bae-2dbfae5f98f5"
-					(reference "R16")
+					(reference "R21")
 					(unit 1)
 				)
@@
 		(on_board yes)
 		(dnp no)
-		(property "Reference" "R20"
+		(property "Reference" "R17"
 			(at 68.58 144.78 90)
 			(effects
@@
 			(project "MX_IMU"
 				(path "/8ed38441-7d4e-4e89-870f-07e11c6dce38/3e6b1080-2480-49a7-8bae-2dbfae5f98f5"
-					(reference "R20")
+					(reference "R17")
 					(unit 1)
 				)
@@
 		(on_board yes)
 		(dnp no)
-		(property "Reference" "R19"
+		(property "Reference" "R16"
 			(at 68.58 138.176 90)
 			(effects
@@
 			(project "MX_IMU"
 				(path "/8ed38441-7d4e-4e89-870f-07e11c6dce38/3e6b1080-2480-49a7-8bae-2dbfae5f98f5"
-					(reference "R19")
+					(reference "R16")
 					(unit 1)
 				)
@@
 		(on_board yes)
 		(dnp no)
-		(property "Reference" "R21"
+		(property "Reference" "R15"
 			(at 53.34 157.48 90)
 			(effects
@@
 			(project "MX_IMU"
 				(path "/8ed38441-7d4e-4e89-870f-07e11c6dce38/3e6b1080-2480-49a7-8bae-2dbfae5f98f5"
-					(reference "R21")
+					(reference "R15")
 					(unit 1)
 				)
@@
 		(on_board yes)
 		(dnp no)
-		(property "Reference" "C30"
+		(property "Reference" "C28"
 			(at 48.4632 151.0284 0)
 			(effects
@@
 			(project "MX_IMU"
 				(path "/8ed38441-7d4e-4e89-870f-07e11c6dce38/3e6b1080-2480-49a7-8bae-2dbfae5f98f5"
-					(reference "C30")
+					(reference "C28")
 					(unit 1)
 				)
@@
 		(on_board yes)
 		(dnp no)
-		(property "Reference" "#PWR078"
+		(property "Reference" "#PWR073"
 			(at 67.31 146.05 0)
 			(effects
@@
 			(project "MX_IMU"
 				(path "/8ed38441-7d4e-4e89-870f-07e11c6dce38/3e6b1080-2480-49a7-8bae-2dbfae5f98f5"
-					(reference "#PWR078")
+					(reference "#PWR073")
 					(unit 1)
 				)
@@
 		(on_board yes)
 		(dnp no)
-		(property "Reference" "#PWR077"
+		(property "Reference" "#PWR074"
 			(at 66.04 147.32 0)
 			(effects
@@
 			(project "MX_IMU"
 				(path "/8ed38441-7d4e-4e89-870f-07e11c6dce38/3e6b1080-2480-49a7-8bae-2dbfae5f98f5"
-					(reference "#PWR077")
+					(reference "#PWR074")
 					(unit 1)
 				)
@@
 		(on_board yes)
 		(dnp no)
-		(property "Reference" "#PWR076"
+		(property "Reference" "#PWR071"
 			(at 50.8 140.97 0)
 			(effects
@@
 			(project "MX_IMU"
 				(path "/8ed38441-7d4e-4e89-870f-07e11c6dce38/3e6b1080-2480-49a7-8bae-2dbfae5f98f5"
-					(reference "#PWR076")
+					(reference "#PWR071")
 					(unit 1)
 				)
@@
 		(dnp no)
 		(fields_autoplaced yes)
-		(property "Reference" "J4"
+		(property "Reference" "J5"
 			(at 128.27 64.7699 0)
 			(effects
@@
 			(project "MX_IMU"
 				(path "/8ed38441-7d4e-4e89-870f-07e11c6dce38/3e6b1080-2480-49a7-8bae-2dbfae5f98f5"
-					(reference "J4")
+					(reference "J5")
 					(unit 1)
 				)
@@
 		(dnp no)
 		(fields_autoplaced yes)
-		(property "Reference" "#PWR074"
+		(property "Reference" "#PWR072"
 			(at 62.23 83.82 0)
 			(effects
@@
 			(project "MX_IMU"
 				(path "/8ed38441-7d4e-4e89-870f-07e11c6dce38/3e6b1080-2480-49a7-8bae-2dbfae5f98f5"
-					(reference "#PWR074")
+					(reference "#PWR072")
 					(unit 1)
 				)
@@
 		(dnp no)
 		(fields_autoplaced yes)
-		(property "Reference" "#PWR071"
+		(property "Reference" "#PWR076"
 			(at 80.01 57.15 0)
 			(effects
@@
 			(project "MX_IMU"
 				(path "/8ed38441-7d4e-4e89-870f-07e11c6dce38/3e6b1080-2480-49a7-8bae-2dbfae5f98f5"
-					(reference "#PWR071")
+					(reference "#PWR076")
 					(unit 1)
 				)
@@
 		(on_board yes)
 		(dnp no)
-		(property "Reference" "#PWR072"
+		(property "Reference" "#PWR070"
 			(at 44.45 68.58 0)
 			(effects
@@
 			(project "MX_IMU"
 				(path "/8ed38441-7d4e-4e89-870f-07e11c6dce38/3e6b1080-2480-49a7-8bae-2dbfae5f98f5"
-					(reference "#PWR072")
+					(reference "#PWR070")
 					(unit 1)
 				)
@@
 		(dnp no)
 		(fields_autoplaced yes)
-		(property "Reference" "J5"
+		(property "Reference" "J4"
 			(at 81.28 142.2399 0)
 			(effects
@@
 			(project "MX_IMU"
 				(path "/8ed38441-7d4e-4e89-870f-07e11c6dce38/3e6b1080-2480-49a7-8bae-2dbfae5f98f5"
-					(reference "J5")
+					(reference "J4")
 					(unit 1)
 				)
@@
 		(on_board yes)
 		(dnp no)
-		(property "Reference" "C29"
+		(property "Reference" "C30"
 			(at 92.71 83.82 0)
 			(effects
@@
 			(project "MX_IMU"
 				(path "/8ed38441-7d4e-4e89-870f-07e11c6dce38/3e6b1080-2480-49a7-8bae-2dbfae5f98f5"
-					(reference "C29")
+					(reference "C30")
 					(unit 1)
 				)
@@
 		(dnp no)
 		(fields_autoplaced yes)
-		(property "Reference" "#PWR070"
+		(property "Reference" "#PWR075"
 			(at 77.47 44.45 0)
 			(effects
@@
 			(project ""
 				(path "/8ed38441-7d4e-4e89-870f-07e11c6dce38/3e6b1080-2480-49a7-8bae-2dbfae5f98f5"
-					(reference "#PWR070")
+					(reference "#PWR075")
 					(unit 1)
 				)
@@
 		(on_board yes)
 		(dnp no)
-		(property "Reference" "R17"
+		(property "Reference" "R18"
 			(at 86.614 73.66 0)
 			(effects
@@
 			(project "MX_IMU"
 				(path "/8ed38441-7d4e-4e89-870f-07e11c6dce38/3e6b1080-2480-49a7-8bae-2dbfae5f98f5"
-					(reference "R17")
+					(reference "R18")
 					(unit 1)
 				)
@@
 		(dnp no)
 		(fields_autoplaced yes)
-		(property "Reference" "#PWR075"
+		(property "Reference" "#PWR077"
 			(at 90.17 96.52 0)
 			(effects
@@
 			(project "MX_IMU"
 				(path "/8ed38441-7d4e-4e89-870f-07e11c6dce38/3e6b1080-2480-49a7-8bae-2dbfae5f98f5"
-					(reference "#PWR075")
+					(reference "#PWR077")
 					(unit 1)
 				)
@@
 		(on_board yes)
 		(dnp no)
-		(property "Reference" "R18"
+		(property "Reference" "R19"
 			(at 96.774 73.66 0)
 			(effects
@@
 			(project "MX_IMU"
 				(path "/8ed38441-7d4e-4e89-870f-07e11c6dce38/3e6b1080-2480-49a7-8bae-2dbfae5f98f5"
-					(reference "R18")
+					(reference "R19")
 					(unit 1)
 				)
@@
 		(on_board yes)
 		(dnp no)
-		(property "Reference" "C28"
+		(property "Reference" "C29"
 			(at 82.55 43.18 0)
 			(effects
@@
 			(project "MX_IMU"
 				(path "/8ed38441-7d4e-4e89-870f-07e11c6dce38/3e6b1080-2480-49a7-8bae-2dbfae5f98f5"
-					(reference "C28")
-					(unit 1)
-				)
+					(reference "C29")
+					(unit 1)
+				)
