File: Connectors.kicad_sch (KiCad schematic)
At the start: 12 parts, among them J4 Conn_02x03_Odd_Even, U12 TJA1051T/3

Commit message: update
Parts:
- added J5: Conn_02x03_Odd_Even, Connector_PinSocket_2.00mm:PinSocket_2x03_P2.00mm_Vertical, symbol Connector_Generic:Conn_02x03_Odd_Even
- TELE1: footprint CONN_SM06B-GHS-TB_JST -> mylib:CONN_SM06B-GHS-TB_JST
Connections:
- net GND: now also J5.2 (Pin_2), J5.4 (Pin_4), J5.6 (Pin_6)
- new net Tim8_2: J5.5 (Pin_5)
- new net Tim8_3: J5.3 (Pin_3)
- new net Tim8_4: J5.1 (Pin_1)
Changed lines of the file:
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@@
+	)
+	(junction
+		(at 219.71 120.65)
+		(diameter 0)
+		(color 0 0 0 0)
 	)
 	(junction
@@
 		(color 0 0 0 0)
 	)
+	(junction
+		(at 219.71 123.19)
+		(diameter 0)
+		(color 0 0 0 0)
+	)
 	(polyline
 		(pts
@@
 	(wire
 		(pts
+			(xy 219.71 123.19) (xy 219.71 125.73)
+		)
+		(stroke
+			(width 0)
+			(type default)
+		)
+	)
+	(wire
+		(pts
 			(xy 80.01 40.64) (xy 80.01 41.91)
 		)
@@
 		(pts
 			(xy 77.47 40.64) (xy 62.23 40.64)
+		)
+		(stroke
+			(width 0)
+			(type default)
+		)
+	)
+	(wire
+		(pts
+			(xy 219.71 120.65) (xy 219.71 123.19)
 		)
 		(stroke
@@
 		)
 	)
+	(global_label "Tim8_4"
+		(shape input)
+		(at 207.01 120.65 180)
+		(effects
+			(font
+				(size 1.27 1.27)
+			)
+			(justify right)
+		)
+		(property "Intersheetrefs" "${INTERSHEET_REFS}"
+			(at 207.01 120.65 0)
+			(effects
+				(font
+					(size 1.27 1.27)
+				)
+				(hide yes)
+			)
+		)
+	)
 	(global_label "SWDIO"
 		(shape input)
@@
 		)
 	)
+	(global_label "Tim8_2"
+		(shape input)
+		(at 207.01 125.73 180)
+		(effects
+			(font
+				(size 1.27 1.27)
+			)
+			(justify right)
+		)
+		(property "Intersheetrefs" "${INTERSHEET_REFS}"
+			(at 207.01 125.73 0)
+			(effects
+				(font
+					(size 1.27 1.27)
+				)
+				(hide yes)
+			)
+		)
+	)
 	(global_label "GPS_RX"
 		(shape input)
@@
 		)
 	)
+	(global_label "Tim8_3"
+		(shape input)
+		(at 207.01 123.19 180)
+		(effects
+			(font
+				(size 1.27 1.27)
+			)
+			(justify right)
+		)
+		(property "Intersheetrefs" "${INTERSHEET_REFS}"
+			(at 207.01 123.19 0)
+			(effects
+				(font
+					(size 1.27 1.27)
+				)
+				(hide yes)
+			)
+		)
+	)
 	(symbol
 		(lib_id "power:GND")
@@
 			)
 		)
-		(property "Footprint" "CONN_SM06B-GHS-TB_JST"
+		(property "Footprint" "mylib:CONN_SM06B-GHS-TB_JST"
 			(at 242.57 78.74 0)
 			(effects
@@
 	)
 	(symbol
+		(lib_id "power:GND")
+		(at 219.71 120.65 180)
+		(unit 1)
+		(exclude_from_sim no)
+		(in_bom yes)
+		(on_board yes)
+		(dnp no)
+		(property "Reference" "#PWR015"
+			(at 219.71 114.3 0)
+			(effects
+				(font
+					(size 1.27 1.27)
+				)
+				(hide yes)
+			)
+		)
+		(property "Value" "GND"
+			(at 219.583 116.2558 0)
+			(effects
+				(font
+					(size 1.27 1.27)
+				)
+			)
+		)
+		(property "Footprint" ""
+			(at 219.71 120.65 0)
+			(effects
+				(font
+					(size 1.27 1.27)
+				)
+				(hide yes)
+			)
+		)
+		(property "Datasheet" ""
+			(at 219.71 120.65 0)
+			(effects
+				(font
+					(size 1.27 1.27)
+				)
+				(hide yes)
+			)
+		)
+		(property "Description" "Power symbol creates a global label with name \"GND\" , ground"
+			(at 219.71 120.65 0)
+			(effects
+				(font
+					(size 1.27 1.27)
+				)
+				(hide yes)
+			)
+		)
+		(pin "1"
+		)
+		(instances
+			(project "MX_IMU"
+				(path "/8ed38441-7d4e-4e89-870f-07e11c6dce38/3e6b1080-2480-49a7-8bae-2dbfae5f98f5"
+					(reference "#PWR015")
+					(unit 1)
+				)
+			)
+		)
+	)
+	(symbol
 		(lib_id "power:+5V")
 		(at 201.93 58.42 0)
@@
 					(unit 1)
 				)
+			)
+		)
+	)
+	(symbol
+		(lib_id "Connector_Generic:Conn_02x03_Odd_Even")
+		(at 212.09 123.19 0)
+		(unit 1)
+		(exclude_from_sim no)
+		(in_bom yes)
+		(on_board yes)
+		(dnp no)
+		(property "Reference" "J5"
+			(at 220.98 116.84 0)
+			(effects
+				(font
+					(size 1.27 1.27)
+				)
+			)
+		)
+		(property "Value" "Conn_02x03_Odd_Even"
+			(at 213.36 116.84 0)
+			(effects
+				(font
+					(size 1.27 1.27)
+				)
+				(hide yes)
+			)
+		)
+		(property "Footprint" "Connector_PinSocket_2.00mm:PinSocket_2x03_P2.00mm_Vertical"
+			(at 212.09 123.19 0)
+			(effects
+				(font
+					(size 1.27 1.27)
+				)
+				(hide yes)
+			)
+		)
+		(property "Datasheet" "~"
+			(at 212.09 123.19 0)
+			(effects
+				(font
+					(size 1.27 1.27)
+				)
+				(hide yes)
+			)
+		)
+		(property "Description" "Generic connector, double row, 02x03, odd/even pin numbering scheme (row 1 odd numbers, row 2 even numbers), script generated (kicad-library-utils/schlib/autogen/connector/)"
+			(at 212.09 123.19 0)
+			(effects
+				(font
+					(size 1.27 1.27)
+				)
+				(hide yes)
+			)
+		)
+		(pin "6"
+		)
+		(pin "1"
+		)
+		(pin "4"
+		)
+		(pin "3"
+		)
+		(pin "2"
+		)
+		(pin "5"
+		)
+		(instances
+			(project "MX_IMU"
+				(path "/8ed38441-7d4e-4e89-870f-07e11c6dce38/3e6b1080-2480-49a7-8bae-2dbfae5f98f5"
+					(reference "J5")
+					(unit 1)
+				)

Commit message: update
Connections:
- net +5V: now also CAN1.1; no longer CAN1.4
- net GND: now also CAN1.4; no longer CAN1.1
Changed lines of the file:
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@@
 	(symbol
 		(lib_id "power:GND")
-		(at 109.22 63.5 180)
+		(at 109.22 73.66 0)
 		(unit 1)
 		(exclude_from_sim no)
@@
 		(dnp no)
 		(property "Reference" "#PWR089"
-			(at 109.22 57.15 0)
+			(at 109.22 80.01 0)
 			(effects
 				(font
@@
 		)
 		(property "Value" "GND"
-			(at 109.093 59.1058 0)
+			(at 109.347 78.0542 0)
 			(effects
 				(font
@@
 		)
 		(property "Footprint" ""
-			(at 109.22 63.5 0)
+			(at 109.22 73.66 0)
 			(effects
 				(font
@@
 		)
 		(property "Datasheet" ""
-			(at 109.22 63.5 0)
+			(at 109.22 73.66 0)
 			(effects
 				(font
@@
 		)
 		(property "Description" "Power symbol creates a global label with name \"GND\" , ground"
-			(at 109.22 63.5 0)
+			(at 109.22 73.66 0)
 			(effects
 				(font
@@
 	(symbol
 		(lib_id "power:+5V")
-		(at 109.22 73.66 180)
+		(at 109.22 63.5 0)
 		(unit 1)
 		(exclude_from_sim no)
@@
 		(dnp no)
 		(property "Reference" "#PWR093"
-			(at 109.22 69.85 0)
+			(at 109.22 67.31 0)
 			(effects
 				(font
@@
 		)
 		(property "Value" "+5V"
-			(at 112.776 77.47 0)
+			(at 105.664 59.69 0)
 			(effects
 				(font
@@
 		)
 		(property "Footprint" ""
-			(at 109.22 73.66 0)
+			(at 109.22 63.5 0)
 			(effects
 				(font
@@
 		)
 		(property "Datasheet" ""
-			(at 109.22 73.66 0)
+			(at 109.22 63.5 0)
 			(effects
 				(font
@@
 		)
 		(property "Description" "Power symbol creates a global label with name \"+5V\""
-			(at 109.22 73.66 0)
-			(effects
-				(font
+			(at 109.22 63.5 0)
+			(effects
+				(font

Commit message: update
Parts:
- renumbered J4 to J5, J5 to J6, R18 to R16, R19 to R17, R20 to R18, R16 to R19, R17 to R20
Changed lines of the file:
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@@
 		(on_board yes)
 		(dnp no)
-		(property "Reference" "#PWR089"
+		(property "Reference" "#PWR090"
 			(at 109.22 80.01 0)
 			(effects
@@
 			(project "MX_IMU"
 				(path "/8ed38441-7d4e-4e89-870f-07e11c6dce38/3e6b1080-2480-49a7-8bae-2dbfae5f98f5"
-					(reference "#PWR089")
+					(reference "#PWR090")
 					(unit 1)
 				)
@@
 		(on_board yes)
 		(dnp no)
-		(property "Reference" "R20"
+		(property "Reference" "R18"
 			(at 73.66 144.78 90)
 			(effects
@@
 			(project "MX_IMU"
 				(path "/8ed38441-7d4e-4e89-870f-07e11c6dce38/3e6b1080-2480-49a7-8bae-2dbfae5f98f5"
-					(reference "R20")
+					(reference "R18")
 					(unit 1)
 				)
@@
 		(on_board yes)
 		(dnp no)
-		(property "Reference" "R19"
+		(property "Reference" "R17"
 			(at 73.66 146.304 90)
 			(effects
@@
 			(project "MX_IMU"
 				(path "/8ed38441-7d4e-4e89-870f-07e11c6dce38/3e6b1080-2480-49a7-8bae-2dbfae5f98f5"
-					(reference "R19")
+					(reference "R17")
 					(unit 1)
 				)
@@
 		(on_board yes)
 		(dnp no)
-		(property "Reference" "R18"
+		(property "Reference" "R16"
 			(at 48.768 142.748 90)
 			(effects
@@
 			(project "MX_IMU"
 				(path "/8ed38441-7d4e-4e89-870f-07e11c6dce38/3e6b1080-2480-49a7-8bae-2dbfae5f98f5"
-					(reference "R18")
+					(reference "R16")
 					(unit 1)
 				)
@@
 		(on_board yes)
 		(dnp no)
-		(property "Reference" "#PWR0100"
+		(property "Reference" "#PWR084"
 			(at 62.23 147.32 0)
 			(effects
@@
 			(project "MX_IMU"
 				(path "/8ed38441-7d4e-4e89-870f-07e11c6dce38/3e6b1080-2480-49a7-8bae-2dbfae5f98f5"
-					(reference "#PWR0100")
+					(reference "#PWR084")
 					(unit 1)
 				)
@@
 		(on_board yes)
 		(dnp no)
-		(property "Reference" "#PWR099"
+		(property "Reference" "#PWR083"
 			(at 52.07 142.24 0)
 			(effects
@@
 			(project "MX_IMU"
 				(path "/8ed38441-7d4e-4e89-870f-07e11c6dce38/3e6b1080-2480-49a7-8bae-2dbfae5f98f5"
-					(reference "#PWR099")
+					(reference "#PWR083")
 					(unit 1)
 				)
@@
 		(dnp no)
 		(fields_autoplaced yes)
-		(property "Reference" "#PWR094"
+		(property "Reference" "#PWR085"
 			(at 62.23 83.82 0)
 			(effects
@@
 			(project "MX_IMU"
 				(path "/8ed38441-7d4e-4e89-870f-07e11c6dce38/3e6b1080-2480-49a7-8bae-2dbfae5f98f5"
-					(reference "#PWR094")
+					(reference "#PWR085")
 					(unit 1)
 				)
@@
 		(dnp no)
 		(fields_autoplaced yes)
-		(property "Reference" "#PWR086"
+		(property "Reference" "#PWR087"
 			(at 80.01 57.15 0)
 			(effects
@@
 			(project "MX_IMU"
 				(path "/8ed38441-7d4e-4e89-870f-07e11c6dce38/3e6b1080-2480-49a7-8bae-2dbfae5f98f5"
-					(reference "#PWR086")
+					(reference "#PWR087")
 					(unit 1)
 				)
@@
 		(on_board yes)
 		(dnp no)
-		(property "Reference" "#PWR092"
+		(property "Reference" "#PWR082"
 			(at 44.45 68.58 0)
 			(effects
@@
 			(project "MX_IMU"
 				(path "/8ed38441-7d4e-4e89-870f-07e11c6dce38/3e6b1080-2480-49a7-8bae-2dbfae5f98f5"
-					(reference "#PWR092")
+					(reference "#PWR082")
 					(unit 1)
 				)
@@
 		(on_board yes)
 		(dnp no)
-		(property "Reference" "#PWR095"
+		(property "Reference" "#PWR096"
 			(at 242.57 72.39 0)
 			(effects
@@
 			(project "MX_IMU"
 				(path "/8ed38441-7d4e-4e89-870f-07e11c6dce38/3e6b1080-2480-49a7-8bae-2dbfae5f98f5"
-					(reference "#PWR095")
+					(reference "#PWR096")
 					(unit 1)
 				)
@@
 		(on_board yes)
 		(dnp no)
-		(property "Reference" "#PWR088"
+		(property "Reference" "#PWR094"
 			(at 226.06 60.96 0)
 			(effects
@@
 			(project "MX_IMU"
 				(path "/8ed38441-7d4e-4e89-870f-07e11c6dce38/3e6b1080-2480-49a7-8bae-2dbfae5f98f5"
-					(reference "#PWR088")
+					(reference "#PWR094")
 					(unit 1)
 				)
@@
 		(dnp no)
 		(fields_autoplaced yes)
-		(property "Reference" "#PWR085"
+		(property "Reference" "#PWR086"
 			(at 77.47 44.45 0)
 			(effects
@@
 			(project ""
 				(path "/8ed38441-7d4e-4e89-870f-07e11c6dce38/3e6b1080-2480-49a7-8bae-2dbfae5f98f5"
-					(reference "#PWR085")
+					(reference "#PWR086")
 					(unit 1)
 				)
@@
 		(on_board yes)
 		(dnp no)
-		(property "Reference" "R16"
+		(property "Reference" "R19"
 			(at 86.614 73.66 0)
 			(effects
@@
 			(project "MX_IMU"
 				(path "/8ed38441-7d4e-4e89-870f-07e11c6dce38/3e6b1080-2480-49a7-8bae-2dbfae5f98f5"
-					(reference "R16")
+					(reference "R19")
 					(unit 1)
 				)
@@
 		(dnp no)
 		(fields_autoplaced yes)
-		(property "Reference" "#PWR097"
+		(property "Reference" "#PWR088"
 			(at 90.17 96.52 0)
 			(effects
@@
 			(project "MX_IMU"
 				(path "/8ed38441-7d4e-4e89-870f-07e11c6dce38/3e6b1080-2480-49a7-8bae-2dbfae5f98f5"
-					(reference "#PWR097")
+					(reference "#PWR088")
 					(unit 1)
 				)
@@
 		(on_board yes)
 		(dnp no)
-		(property "Reference" "R17"
+		(property "Reference" "R20"
 			(at 96.774 73.66 0)
 			(effects
@@
 			(project "MX_IMU"
 				(path "/8ed38441-7d4e-4e89-870f-07e11c6dce38/3e6b1080-2480-49a7-8bae-2dbfae5f98f5"
-					(reference "R17")
+					(reference "R20")
 					(unit 1)
 				)
@@
 		(on_board yes)
 		(dnp no)
-		(property "Reference" "J4"
+		(property "Reference" "J5"
 			(at 72.39 138.43 0)
 			(effects
@@
 			(project ""
 				(path "/8ed38441-7d4e-4e89-870f-07e11c6dce38/3e6b1080-2480-49a7-8bae-2dbfae5f98f5"
-					(reference "J4")
+					(reference "J5")
 					(unit 1)
 				)
@@
 		(on_board yes)
 		(dnp no)
-		(property "Reference" "#PWR098"
+		(property "Reference" "#PWR097"
 			(at 242.57 87.63 0)
 			(effects
@@
 			(project "MX_IMU"
 				(path "/8ed38441-7d4e-4e89-870f-07e11c6dce38/3e6b1080-2480-49a7-8bae-2dbfae5f98f5"
-					(reference "#PWR098")
+					(reference "#PWR097")
 					(unit 1)
 				)
@@
 		(on_board yes)
 		(dnp no)
-		(property "Reference" "#PWR093"
+		(property "Reference" "#PWR089"
 			(at 109.22 67.31 0)
 			(effects
@@
 			(project "MX_IMU"
 				(path "/8ed38441-7d4e-4e89-870f-07e11c6dce38/3e6b1080-2480-49a7-8bae-2dbfae5f98f5"
-					(reference "#PWR093")
+					(reference "#PWR089")
 					(unit 1)
 				)
@@
 		(on_board yes)
 		(dnp no)
-		(property "Reference" "#PWR096"
+		(property "Reference" "#PWR098"
 			(at 266.7 82.55 0)
 			(effects
@@
 			(project "MX_IMU"
 				(path "/8ed38441-7d4e-4e89-870f-07e11c6dce38/3e6b1080-2480-49a7-8bae-2dbfae5f98f5"
-					(reference "#PWR096")
+					(reference "#PWR098")
 					(unit 1)
 				)
@@
 		(on_board yes)
 		(dnp no)
-		(property "Reference" "#PWR090"
+		(property "Reference" "#PWR091"
 			(at 133.35 66.04 0)
 			(effects
@@
 			(project "MX_IMU"
 				(path "/8ed38441-7d4e-4e89-870f-07e11c6dce38/3e6b1080-2480-49a7-8bae-2dbfae5f98f5"
-					(reference "#PWR090")
+					(reference "#PWR091")
 					(unit 1)
 				)
@@
 		(on_board yes)
 		(dnp no)
-		(property "Reference" "#PWR015"
+		(property "Reference" "#PWR095"
 			(at 219.71 114.3 0)
 			(effects
@@
 			(project "MX_IMU"
 				(path "/8ed38441-7d4e-4e89-870f-07e11c6dce38/3e6b1080-2480-49a7-8bae-2dbfae5f98f5"
-					(reference "#PWR015")
+					(reference "#PWR095")
 					(unit 1)
 				)
@@
 		(on_board yes)
 		(dnp no)
-		(property "Reference" "#PWR087"
+		(property "Reference" "#PWR092"
 			(at 201.93 62.23 0)
 			(effects
@@
 			(project "MX_IMU"
 				(path "/8ed38441-7d4e-4e89-870f-07e11c6dce38/3e6b1080-2480-49a7-8bae-2dbfae5f98f5"
-					(reference "#PWR087")
+					(reference "#PWR092")
 					(unit 1)
 				)
@@
 		(on_board yes)
 		(dnp no)
-		(property "Reference" "#PWR091"
+		(property "Reference" "#PWR093"
 			(at 201.93 72.39 0)
 			(effects
@@
 			(project "MX_IMU"
 				(path "/8ed38441-7d4e-4e89-870f-07e11c6dce38/3e6b1080-2480-49a7-8bae-2dbfae5f98f5"
-					(reference "#PWR091")
+					(reference "#PWR093")
 					(unit 1)
 				)
@@
 		(on_board yes)
 		(dnp no)
-		(property "Reference" "J5"
+		(property "Reference" "J6"
 			(at 220.98 116.84 0)
 			(effects
@@
 			(project "MX_IMU"
 				(path "/8ed38441-7d4e-4e89-870f-07e11c6dce38/3e6b1080-2480-49a7-8bae-2dbfae5f98f5"
-					(reference "J5")
-					(unit 1)
-				)
+					(reference "J6")
+					(unit 1)
+				)

Commit message: PumbaaV2_RC2
Parts:
- CAN1, GPS_Serial1: value SM04B-GHS-TB -> SM04B-GHS-TB(LF)(SN)
- R19: LCSC Part (none) -> C166918
- R20: LCSC (none) -> C166918
- TELE1: value SM06B-GHS-TB -> SM06B-GHS-TB(LF)(SN)
Other:
- note added: "Additional Connectors"
- moved on the sheet: J6, TELE1
