File: _autosave-MX_IMU.kicad_pcb (KiCad board)
At the start: 4 copper layers, 84 parts, among them J1 S2B-ZRLFSN, J2 Native USB, J3 Native USB, J4 Conn_01x06, J5 Conn_01x06, SW1 SW_Push, U1 CH340E, U10 TJA1051T/3, U2 NCP1117-5.0_SOT223, U3 TPS2115ADRBR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

Commit message: update
Parts:
- moved JP3 130.1 mm to (100.6, 133.3)
- moved SW1 128.1 mm to (88.3, 133.1)
- moved Y1 117.9 mm to (115.2, 115.7)
- moved J1 115.5 mm to (78.6, 89.1)
- moved U1 109.2 mm to (82.7, 74.8)
- moved U2 105.8 mm to (101.1, 76.3)
- moved U3 104.6 mm to (111.6, 74.6)
- moved JP1 101.1 mm to (84.6, 79.8)
- moved U9 92.3 mm to (95.7, 117.6)
- moved U4 86.3 mm to (114.6, 87.1)
- moved U5 78.6 mm to (91.9, 80.8)
- moved JP2 75.2 mm to (121.6, 74.3)
- moved J2 73.0 mm to (92.4, 67.3)
- moved C29 72.1 mm to (119.7, 99.5)
- moved C30 72.1 mm to (116.3, 97.8)
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Other:
- board outline added: 50 x 80 mm
