File: _autosave-MX_IMU.kicad_pcb (KiCad board)
At the start: 4 copper layers, 50 x 80 mm, 84 parts, among them J1 S2B-ZRLFSN, J2 Native USB, J3 Native USB, J5 Conn_01x06, U1 USBLC6-2SC6, U10 TJA1051T/3, U2 NCP1117-5.0_SOT223, U3 ld39150dt33-r, U4 TPS2115ADRBR, U5 USBLC6-2SC6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

Commit message: updateu
Parts:
- moved LED 30.3 mm to (79.6, 128.8)
- moved BOOT0 27.3 mm to (84.1, 127.5), turned to 0 degrees
- renumbered CAN1 to CAN, UART1 to UART
Routing:
- net SWDIO: track 0.97 -> 19.2 mm
- net Net-(J5-Pin_3): track 5.04 -> 2.59 mm
Changed lines of the file:
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@@
 		(layer "F.Cu")
 		(at 118.2491 121.92846 -90)
-		(property "Reference" "UART1"
-			(at -11.1082 -3.948 90)
+		(property "Reference" "UART"
+			(at 4.3918 -4.802 90)
 			(layer "F.SilkS")
 			(effects
@@
 		(fp_text user "353630460"
 			(at -8.1788 -16.002 90)
-			(layer "F.SilkS")
-			(effects
-				(font
-					(size 1 1)
-					(thickness 0.15)
-				)
-			)
-		)
-		(fp_text user "353630460"
-			(at -8.1788 -16.002 90)
 			(layer "F.Fab")
 			(effects
@@
 	(footprint "LED_SMD:LED_WS2812B-2020_PLCC4_2.0x2.0mm"
 		(layer "F.Cu")
-		(at 98.5011 105.23526 90)
+		(at 79.5511 128.82026 90)
 		(descr "2.0mm x 2.0mm Addressable RGB LED NeoPixel Nano, 12 mA, https://cdn-shop.adafruit.com/product-files/4684/4684_WS2812B-2020_V1.3_EN.pdf")
 		(tags "LED RGB NeoPixel Nano PLCC-4 2020")
@@
 		(layer "F.Cu")
 		(at 81.5511 116.33246 90)
-		(property "Reference" "CAN1"
-			(at 4.17974 -3.302 90)
+		(property "Reference" "CAN"
+			(at -9.9878 -4 90)
 			(layer "F.SilkS")
 			(effects
@@
 	(footprint "Connector_PinHeader_2.54mm:PinHeader_1x02_P2.54mm_Vertical"
 		(layer "F.Cu")
-		(at 111.1261 130.93026 180)
+		(at 84.0511 127.54526)
 		(descr "Through hole straight pin header, 1x02, 2.54mm pitch, single row")
 		(tags "Through hole pin header THT 1x02 2.54mm single row")
 		(property "Reference" "BOOT0"
-			(at 0 -2.38 0)
+			(at 2 6.275 0)
 			(layer "F.SilkS")
 			(effects
@@
 		(attr through_hole)
 		(fp_line
-			(start 1.38 1.27)
-			(end 1.38 3.92)
+			(start -1.38 -1.38)
+			(end 0 -1.38)
 			(stroke
 				(width 0.12)
@@
 		)
 		(fp_line
-			(start -1.38 3.92)
-			(end 1.38 3.92)
+			(start -1.38 0)
+			(end -1.38 -1.38)
 			(stroke
 				(width 0.12)
@@
 		(fp_line
 			(start -1.38 1.27)
-			(end 1.38 1.27)
+			(end -1.38 3.92)
 			(stroke
 				(width 0.12)
@@
 		(fp_line
 			(start -1.38 1.27)
-			(end -1.38 3.92)
+			(end 1.38 1.27)
 			(stroke
 				(width 0.12)
@@
 		)
 		(fp_line
-			(start -1.38 0)
-			(end -1.38 -1.38)
+			(start -1.38 3.92)
+			(end 1.38 3.92)
 			(stroke
 				(width 0.12)
@@
 		)
 		(fp_line
-			(start -1.38 -1.38)
-			(end 0 -1.38)
+			(start 1.38 1.27)
+			(end 1.38 3.92)
 			(stroke
 				(width 0.12)
@@
 		)
 		(fp_line
-			(start 1.77 4.32)
-			(end 1.77 -1.77)
+			(start -1.77 -1.77)
+			(end -1.77 4.32)
 			(stroke
 				(width 0.05)
@@
 		)
 		(fp_line
-			(start 1.77 -1.77)
-			(end -1.77 -1.77)
+			(start -1.77 4.32)
+			(end 1.77 4.32)
 			(stroke
 				(width 0.05)
@@
 		)
 		(fp_line
-			(start -1.77 4.32)
-			(end 1.77 4.32)
+			(start 1.77 -1.77)
+			(end -1.77 -1.77)
 			(stroke
 				(width 0.05)
@@
 		)
 		(fp_line
-			(start -1.77 -1.77)
-			(end -1.77 4.32)
+			(start 1.77 4.32)
+			(end 1.77 -1.77)
 			(stroke
 				(width 0.05)
@@
 		)
 		(fp_line
-			(start 1.27 3.81)
-			(end -1.27 3.81)
+			(start -1.27 -0.635)
+			(end -0.635 -1.27)
 			(stroke
 				(width 0.1)
@@
 		)
 		(fp_line
-			(start 1.27 -1.27)
-			(end 1.27 3.81)
+			(start -1.27 3.81)
+			(end -1.27 -0.635)
 			(stroke
 				(width 0.1)
@@
 		)
 		(fp_line
-			(start -1.27 3.81)
-			(end -1.27 -0.635)
+			(start 1.27 -1.27)
+			(end 1.27 3.81)
 			(stroke
 				(width 0.1)
@@
 		)
 		(fp_line
-			(start -1.27 -0.635)
-			(end -0.635 -1.27)
+			(start 1.27 3.81)
+			(end -1.27 3.81)
 			(stroke
 				(width 0.1)
@@
 		)
 		(pad "1" thru_hole rect
-			(at 0 0 180)
+			(at 0 0)
 			(size 1.7 1.7)
 			(drill 1)
@@
 		)
 		(pad "2" thru_hole circle
-			(at 0 2.54 180)
+			(at 0 2.54)
 			(size 1.7 1.7)
 			(drill 1)
@@
 	)
 	(segment
+		(start 99.794278 114.33126)
+		(end 100.0511 114.074438)
+		(width 0.25)
+		(layer "F.Cu")
+		(net 12)
+	)
+	(segment
+		(start 86.5611 108.32026)
+		(end 93.438634 108.32026)
+		(width 0.25)
+		(layer "F.Cu")
+		(net 12)
+	)
+	(segment
+		(start 96.3451 111.226726)
+		(end 96.3451 113.36098)
+		(width 0.25)
+		(layer "F.Cu")
+		(net 12)
+	)
+	(segment
+		(start 100.0511 114.074438)
+		(end 100.0511 113.23026)
+		(width 0.25)
+		(layer "F.Cu")
+		(net 12)
+	)
+	(segment
+		(start 93.438634 108.32026)
+		(end 96.3451 111.226726)
+		(width 0.25)
+		(layer "F.Cu")
+		(net 12)
+	)
+	(segment
+		(start 96.3451 113.36098)
+		(end 97.31538 114.33126)
+		(width 0.25)
+		(layer "F.Cu")
+		(net 12)
+	)
+	(segment
+		(start 97.31538 114.33126)
+		(end 99.794278 114.33126)
+		(width 0.25)
+		(layer "F.Cu")
+		(net 12)
+	)
+	(segment
 		(start 100.0511 113.23026)
 		(end 100.0271 113.23026)
@@
 	)
 	(segment
-		(start 85.5911 110.82026)
-		(end 85.5911 113.27026)
-		(width 0.25)
-		(layer "F.Cu")
-		(net 60)
-	)
-	(segment
