File: _autosave-MX_IMU.kicad_pcb (KiCad board)
At the start: 4 copper layers, 50 x 80 mm, 83 parts, among them J1 B2B-PH-K-S, J2 Native USB, J3 Native USB, J4 Conn_02x03_Odd_Even, SW1 SSSS213000, SW2 SSSS213000, U1 USBLC6-2SC6, U10 ICM-42688-P, U11 W25Q128JVS, U12 TJA1051T/3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

Commit message: update
Routing:
- net GND: track 151.7 -> 161.2 mm, vias 57 -> 59
- net Serial_D-: track 0.00 -> 3.28 mm
- net VBUS: track 13.5 -> 10.7 mm
- net Serial_VBUS: track 32.8 -> 35.1 mm
- net +5VD: vias 4 -> 2
