File: MCU.kicad_sch (KiCad schematic)
At the start: 24 parts, among them U1 STM32F405RGT6, Y1 16MHz

Commit message: update
Parts:
- removed H1, H2, H3, H4: MountingHole_Pad, MountingHole:MountingHole_3.2mm_M3_Pad_Via, symbol Mechanical:MountingHole_Pad
- added C26: 100nf, Capacitor_SMD:C_0603_1608Metric, symbol Device:C_Small
- added JP3: N_USB_VBUS, Connector_PinHeader_2.54mm:PinHeader_1x02_P2.54mm_Vertical, symbol Jumper:Jumper_2_Open
- added SW1: RESET, Button_Switch_THT:SW_PUSH_6mm, symbol Switch:SW_Push
- renumbered C1 to C10, C4 to C11, C5 to C12, C6 to C13, C7 to C14, C8 to C15, C9 to C16, C10 to C17, C13 to C18, C11 to C19, C12 to C20, C2 to C21, C3 to C22, D1 to D4, R3 to R10, R2 to R11, R1 to R9, U1 to U7
Connections:
- net +3.3V: now also JP3.1 (A)
- net BOOT0: now also JP3.2 (B)
- net GND: now also C26.1, SW1.2
- net NRST: now also C26.2, SW1.1
Other:
- removed sheet Connectors
- removed sheet PowerSupply
- note added: "Reset Switch"
- note removed: "Mounting Holes"
- title: STM32_Sensor_MX -> (none)
- moved on the sheet: C10, C11, C12, C13, C14, C15, C16, C17, C18, C19, C20, C21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

Commit message: update
Connections:
- net CAN2_RX: now also U7.57 (PB5); no longer U7.33 (PB12)
- net CAN2_TX: now also U7.58 (PB6); no longer U7.34 (PB13)
- net Status_LED: now also U7.30 (PB11); no longer U7.57 (PB5)
- net Flash_MISO: now reaches U7.35 (PB14)
- net Flash_MOSI: now reaches U7.36 (PB15)
- net Flash_CS: now reaches U7.37 (PC6)
- new net Flash_CLK: U7.34 (PB13)
- no-connect marks 32 -> 28
Changed lines of the file:
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@@
-	)
-	(no_connect
-		(at 102.87 172.72)
 	)
 	(no_connect
@@
 	)
 	(no_connect
+		(at 102.87 165.1)
+	)
+	(no_connect
 		(at 62.23 152.4)
 	)
@@
 	)
 	(no_connect
-		(at 102.87 162.56)
-	)
-	(no_connect
 		(at 102.87 111.76)
 	)
@@
 	)
 	(no_connect
-		(at 105.41 149.86)
-	)
-	(no_connect
-		(at 62.23 129.54)
-	)
-	(no_connect
 		(at 102.87 93.98)
 	)
 	(no_connect
-		(at 102.87 170.18)
-	)
-	(no_connect
 		(at 102.87 154.94)
 	)
@@
 	(wire
 		(pts
-			(xy 102.87 147.32) (xy 105.41 147.32)
-		)
-		(stroke
-			(width 0)
-			(type default)
-		)
-	)
-	(wire
-		(pts
 			(xy 80.01 53.34) (xy 90.17 53.34)
 		)
@@
 		(pts
 			(xy 82.55 181.61) (xy 82.55 180.34)
-		)
-		(stroke
-			(width 0)
-			(type default)
-		)
-	)
-	(wire
-		(pts
-			(xy 102.87 149.86) (xy 105.41 149.86)
 		)
 		(stroke
@@
 		)
 	)
+	(global_label "CAN2_TX"
+		(shape input)
+		(at 102.87 149.86 0)
+		(effects
+			(font
+				(size 1.27 1.27)
+			)
+			(justify left)
+		)
+		(property "Intersheetrefs" "${INTERSHEET_REFS}"
+			(at 102.87 149.86 0)
+			(effects
+				(font
+					(size 1.27 1.27)
+				)
+				(hide yes)
+			)
+		)
+	)
 	(global_label "HSE_OUT"
 		(shape input)
@@
 		)
 	)
+	(global_label "GYRO_CS"
+		(shape input)
+		(at 62.23 124.46 180)
+		(effects
+			(font
+				(size 1.27 1.27)
+			)
+			(justify right)
+		)
+		(property "Intersheetrefs" "${INTERSHEET_REFS}"
+			(at 62.23 124.46 0)
+			(effects
+				(font
+					(size 1.27 1.27)
+				)
+				(hide yes)
+			)
+		)
+	)
+	(global_label "SWCLK"
+		(shape input)
+		(at 105.41 127 0)
+		(effects
+			(font
+				(size 1.27 1.27)
+			)
+			(justify left)
+		)
+		(property "Intersheetrefs" "${INTERSHEET_REFS}"
+			(at 105.41 127 0)
+			(effects
+				(font
+					(size 1.27 1.27)
+				)
+				(hide yes)
+			)
+		)
+	)
 	(global_label "CAN2_RX"
 		(shape input)
-		(at 102.87 165.1 0)
-		(effects
-			(font
-				(size 1.27 1.27)
-			)
-			(justify left)
-		)
-		(property "Intersheetrefs" "${INTERSHEET_REFS}"
-			(at 102.87 165.1 0)
-			(effects
-				(font
-					(size 1.27 1.27)
-				)
-				(hide yes)
-			)
-		)
-	)
-	(global_label "GYRO_CS"
-		(shape input)
-		(at 62.23 124.46 180)
-		(effects
-			(font
-				(size 1.27 1.27)
-			)
-			(justify right)
-		)
-		(property "Intersheetrefs" "${INTERSHEET_REFS}"
-			(at 62.23 124.46 0)
-			(effects
-				(font
-					(size 1.27 1.27)
-				)
-				(hide yes)
-			)
-		)
-	)
-	(global_label "SWCLK"
-		(shape input)
-		(at 105.41 127 0)
-		(effects
-			(font
-				(size 1.27 1.27)
-			)
-			(justify left)
-		)
-		(property "Intersheetrefs" "${INTERSHEET_REFS}"
-			(at 105.41 127 0)
+		(at 102.87 147.32 0)
+		(effects
+			(font
+				(size 1.27 1.27)
+			)
+			(justify left)
+		)
+		(property "Intersheetrefs" "${INTERSHEET_REFS}"
+			(at 102.87 147.32 0)
 			(effects
 				(font
@@
 		)
 	)
-	(global_label "CAN2_TX"
+	(global_label "Flash_CLK"
 		(shape input)
 		(at 102.87 167.64 0)
-		(effects
-			(font
-				(size 1.27 1.27)
-			)
-			(justify left)
-		)
-		(property "Intersheetrefs" "${INTERSHEET_REFS}"
-			(at 102.87 167.64 0)
-			(effects
-				(font
-					(size 1.27 1.27)
-				)
+		(fields_autoplaced yes)
+		(effects
+			(font
+				(size 1.27 1.27)
+			)
+			(justify left)
+		)
+		(property "Intersheetrefs" "${INTERSHEET_REFS}"
+			(at 115.4708 167.64 0)
+			(effects
+				(font
+					(size 1.27 1.27)
+				)
+				(justify left)
 				(hide yes)
 			)
@@
 	(global_label "Status_LED"
 		(shape input)
-		(at 105.41 147.32 0)
+		(at 102.87 162.56 0)
 		(fields_autoplaced yes)
 		(effects
@@
 		)
 		(property "Intersheetrefs" "${INTERSHEET_REFS}"
-			(at 118.7969 147.32 0)
+			(at 116.2569 162.56 0)
 			(effects
 				(font
@@
 		)
 	)
+	(global_label "Flash_CS"
+		(shape input)
+		(at 62.23 129.54 180)
+		(fields_autoplaced yes)
+		(effects
+			(font
+				(size 1.27 1.27)
+			)
+			(justify right)
+		)
+		(property "Intersheetrefs" "${INTERSHEET_REFS}"
+			(at 50.7178 129.54 0)
+			(effects
+				(font
+					(size 1.27 1.27)
+				)
+				(justify right)
+				(hide yes)
+			)
+		)
+	)
 	(global_label "HSE_OUT"
 		(shape input)
@@
 					(size 1.27 1.27)
 				)
+				(hide yes)
+			)
+		)
+	)
+	(global_label "Flash_MISO"
+		(shape input)
+		(at 102.87 170.18 0)
+		(fields_autoplaced yes)
+		(effects
+			(font
+				(size 1.27 1.27)
+			)
+			(justify left)
+		)
+		(property "Intersheetrefs" "${INTERSHEET_REFS}"
+			(at 116.4989 170.18 0)
+			(effects
+				(font
+					(size 1.27 1.27)
+				)
+				(justify left)
 				(hide yes)
 			)
@@
 				(hide yes)
 			)
+		)
+	)
+	(global_label "Flash_MOSI"
+		(shape input)
+		(at 102.87 172.72 0)
+		(fields_autoplaced yes)
+		(effects
+			(font
+				(size 1.27 1.27)
+			)
+			(justify left)
+		)
+		(property "Intersheetrefs" "${INTERSHEET_REFS}"
+			(at 116.4989 172.72 0)
+			(effects
+				(font
+					(size 1.27 1.27)
+				)
+				(justify left)
+				(hide yes)
+			)

Commit message: update spi flash and ws2812b
Parts:
- removed D4: WS2812, LED_SMD:LED_WS2812_PLCC6_5.0x5.0mm_P1.6mm, symbol LED:WS2812
- added D5: WS2812B-2020, LED_SMD:LED_WS2812B-2020_PLCC4_2.0x2.0mm, symbol LED:WS2812B-2020
Connections:
- net +5V: now also D5.4 (VDD)
- net GND: now also D5.2 (VSS)
- net Status_LED: now also D5.3 (DIN)
Other:
- note added: "need replace LED with ws2812B"
Changed lines of the file:
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@@
 	(generator_version "9.0")
 	(paper "A4")
+	(text "need replace LED with ws2812B"
+		(exclude_from_sim no)
+		(at 246.888 77.47 0)
+		(effects
+			(font
+				(size 1.27 1.27)
+			)
+		)
+	)
 	(text "HSE"
 		(exclude_from_sim no)
@@
 	)
 	(junction
-		(at 229.87 88.9)
-		(diameter 0)
-		(color 0 0 0 0)
-	)
-	(junction
 		(at 154.94 148.59)
 		(diameter 0)
@@
 	(wire
 		(pts
-			(xy 227.33 88.9) (xy 229.87 88.9)
-		)
-		(stroke
-			(width 0)
-			(type default)
-		)
-	)
-	(wire
-		(pts
 			(xy 102.87 127) (xy 105.41 127)
 		)
@@
 	)
 	(symbol
+		(lib_id "LED:WS2812B-2020")
+		(at 229.87 96.52 0)
+		(unit 1)
+		(exclude_from_sim no)
+		(in_bom yes)
+		(on_board yes)
+		(dnp no)
+		(fields_autoplaced yes)
+		(property "Reference" "D5"
+			(at 243.84 90.0998 0)
+			(effects
+				(font
+					(size 1.27 1.27)
+				)
+			)
+		)
+		(property "Value" "WS2812B-2020"
+			(at 243.84 92.6398 0)
+			(effects
+				(font
+					(size 1.27 1.27)
+				)
+			)
+		)
+		(property "Footprint" "LED_SMD:LED_WS2812B-2020_PLCC4_2.0x2.0mm"
+			(at 231.14 104.14 0)
+			(effects
+				(font
+					(size 1.27 1.27)
+				)
+				(justify left top)
+				(hide yes)
+			)
+		)
+		(property "Datasheet" "https://cdn-shop.adafruit.com/product-files/4684/4684_WS2812B-2020_V1.3_EN.pdf"
+			(at 232.41 106.045 0)
+			(effects
+				(font
+					(size 1.27 1.27)
+				)
+				(justify left top)
+				(hide yes)
+			)
+		)
+		(property "Description" "RGB LED with integrated controller, 2.0 x 2.0 mm, 12 mA"
+			(at 229.87 96.52 0)
+			(effects
+				(font
+					(size 1.27 1.27)
+				)
+				(hide yes)
+			)
+		)
+		(pin "3"
+		)
+		(pin "1"
+		)
+		(pin "2"
+		)
+		(pin "4"
+		)
+		(instances
+			(project ""
+				(path "/8ed38441-7d4e-4e89-870f-07e11c6dce38/39c93069-edc2-4035-8fc7-27a45736847d"
+					(reference "D5")
+					(unit 1)
+				)
+			)
+		)
+	)
+	(symbol
 		(lib_id "power:+5V")
 		(at 229.87 86.36 0)
@@
 					(unit 1)
 				)
-			)
-		)
-	)
-	(symbol
-		(lib_id "LED:WS2812")
-		(at 229.87 96.52 0)
-		(unit 1)
-		(exclude_from_sim no)
-		(in_bom yes)
-		(on_board yes)
-		(dnp no)
-		(fields_autoplaced yes)
-		(property "Reference" "D4"
-			(at 239.5409 93.0616 0)
-			(effects
-				(font
-					(size 1.27 1.27)
-				)
-			)
-		)
-		(property "Value" "WS2812"
-			(at 239.5409 95.5985 0)
-			(effects
-				(font
-					(size 1.27 1.27)
-				)
-			)
-		)
-		(property "Footprint" "LED_SMD:LED_WS2812_PLCC6_5.0x5.0mm_P1.6mm"
-			(at 231.14 104.14 0)
-			(effects
-				(font
-					(size 1.27 1.27)
-				)
-				(justify left top)
-				(hide yes)
-			)
-		)
-		(property "Datasheet" "https://cdn-shop.adafruit.com/datasheets/WS2812.pdf"
-			(at 232.41 106.045 0)
-			(effects
-				(font
-					(size 1.27 1.27)
-				)
-				(justify left top)
-				(hide yes)
-			)
-		)
-		(property "Description" ""
-			(at 229.87 96.52 0)
-			(effects
-				(font
-					(size 1.27 1.27)
-				)
-			)
-		)
-		(pin "1"
-		)
-		(pin "2"
-		)
-		(pin "3"
-		)
-		(pin "4"
-		)
-		(pin "5"
-		)
-		(pin "6"
-		)
-		(instances
-			(project "MX_IMU"
-				(path "/8ed38441-7d4e-4e89-870f-07e11c6dce38/39c93069-edc2-4035-8fc7-27a45736847d"
-					(reference "D4")
-					(unit 1)
-				)

Commit message: update library
Parts:
- C10: value 4u7 -> C_Small
- C11, C12, C13, C14, C15: value 100n -> C_Small
- C16: value 1u -> C_Small
- C17: value 10n -> C_Small
- C18: value 100nf -> C_Small
- C19, C20: value 12p -> C_Small
- C21: renamed from C26; value 100nf -> C_Small
- C22: renamed from C21; value 2u2 -> C_Small
- C23: renamed from C22; value 2u2 -> C_Small
- FB1: value 600 @ 600 MHz -> FerriteBead_Small
- JP3: value N_USB_VBUS -> Jumper_2_Open
- R10: value 10k -> R_Small
- R11: value 10k -> R
- R9: value 47 -> R_Small
- SW1: value RESET -> SW_Push
- U7: value STM32F405RGT6 -> STM32F405RGTx
- Y1: value 16MHz -> Crystal_GND24_Small
- renumbered D5 to D4
Changed lines of the file:
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@@
 			)
 		)
-		(property "Value" "STM32F405RGT6"
+		(property "Value" "STM32F405RGTx"
 			(at 94.615 176.53 0)
 			(effects
@@
 		(on_board yes)
 		(dnp no)
-		(property "Reference" "#PWR058"
+		(property "Reference" "#PWR059"
 			(at 85.09 189.23 0)
 			(effects
@@
 			(project "MX_IMU"
 				(path "/8ed38441-7d4e-4e89-870f-07e11c6dce38/39c93069-edc2-4035-8fc7-27a45736847d"
-					(reference "#PWR058")
+					(reference "#PWR059")
 					(unit 1)
 				)
@@
 		(on_board yes)
 		(dnp no)
-		(property "Reference" "#PWR050"
+		(property "Reference" "#PWR046"
 			(at 77.47 85.09 0)
 			(effects
@@
 			(project "MX_IMU"
 				(path "/8ed38441-7d4e-4e89-870f-07e11c6dce38/39c93069-edc2-4035-8fc7-27a45736847d"
-					(reference "#PWR050")
+					(reference "#PWR046")
 					(unit 1)
 				)
@@
 		(on_board yes)
 		(dnp no)
-		(property "Reference" "#PWR051"
+		(property "Reference" "#PWR047"
 			(at 90.17 85.09 0)
 			(effects
@@
 			(project "MX_IMU"
 				(path "/8ed38441-7d4e-4e89-870f-07e11c6dce38/39c93069-edc2-4035-8fc7-27a45736847d"
-					(reference "#PWR051")
+					(reference "#PWR047")
 					(unit 1)
 				)
@@
 		(on_board yes)
 		(dnp no)
-		(property "Reference" "C22"
+		(property "Reference" "C23"
 			(at 62.23 166.37 0)
 			(effects
@@
 			)
 		)
-		(property "Value" "2u2"
+		(property "Value" "C_Small"
 			(at 62.23 168.91 0)
 			(effects
@@
 			(project "MX_IMU"
 				(path "/8ed38441-7d4e-4e89-870f-07e11c6dce38/39c93069-edc2-4035-8fc7-27a45736847d"
-					(reference "C22")
+					(reference "C23")
 					(unit 1)
 				)
@@
 		(on_board yes)
 		(dnp no)
-		(property "Reference" "C21"
+		(property "Reference" "C22"
 			(at 54.61 161.29 0)
 			(effects
@@
 			)
 		)
-		(property "Value" "2u2"
+		(property "Value" "C_Small"
 			(at 54.61 163.83 0)
 			(effects
@@
 			(project "MX_IMU"
 				(path "/8ed38441-7d4e-4e89-870f-07e11c6dce38/39c93069-edc2-4035-8fc7-27a45736847d"
-					(reference "C21")
+					(reference "C22")
 					(unit 1)
 				)
@@
 		(on_board yes)
 		(dnp no)
-		(property "Reference" "#PWR057"
+		(property "Reference" "#PWR058"
 			(at 59.69 177.8 0)
 			(effects
@@
 			(project "MX_IMU"
 				(path "/8ed38441-7d4e-4e89-870f-07e11c6dce38/39c93069-edc2-4035-8fc7-27a45736847d"
-					(reference "#PWR057")
+					(reference "#PWR058")
 					(unit 1)
 				)
@@
 		(on_board yes)
 		(dnp no)
-		(property "Reference" "#PWR056"
+		(property "Reference" "#PWR057"
 			(at 52.07 171.45 0)
 			(effects
@@
 			(project "MX_IMU"
 				(path "/8ed38441-7d4e-4e89-870f-07e11c6dce38/39c93069-edc2-4035-8fc7-27a45736847d"
-					(reference "#PWR056")
+					(reference "#PWR057")
 					(unit 1)
 				)
@@
 			)
 		)
-		(property "Value" "4u7"
+		(property "Value" "C_Small"
 			(at 53.34 50.8 0)
 			(effects
@@
 			)
 		)
-		(property "Value" "100n"
+		(property "Value" "C_Small"
 			(at 62.23 50.8 0)
 			(effects
@@
 			)
 		)
-		(property "Value" "100n"
+		(property "Value" "C_Small"
 			(at 72.39 50.8 0)
 			(effects
@@
 			)
 		)
-		(property "Value" "100n"
+		(property "Value" "C_Small"
 			(at 82.55 50.8 0)
 			(effects
@@
 			)
 		)
-		(property "Value" "100n"
+		(property "Value" "C_Small"
 			(at 92.71 50.8 0)
 			(effects
@@
 			)
 		)
-		(property "Value" "100n"
+		(property "Value" "C_Small"
 			(at 102.87 50.8 0)
 			(effects
@@
 		(on_board yes)
 		(dnp no)
-		(property "Reference" "#PWR046"
+		(property "Reference" "#PWR044"
 			(at 50.8 60.96 0)
 			(effects
@@
 			(project "MX_IMU"
 				(path "/8ed38441-7d4e-4e89-870f-07e11c6dce38/39c93069-edc2-4035-8fc7-27a45736847d"
-					(reference "#PWR046")
+					(reference "#PWR044")
 					(unit 1)
 				)
@@
 			)
 		)
-		(property "Value" "600 @ 600 MHz"
+		(property "Value" "FerriteBead_Small"
 			(at 127 50.165 90)
 			(effects
@@
 			)
 		)
-		(property "Value" "1u"
+		(property "Value" "C_Small"
 			(at 139.7 52.07 0)
 			(effects
@@
 			)
 		)
-		(property "Value" "10n"
+		(property "Value" "C_Small"
 			(at 151.13 52.07 0)
 			(effects
@@
 		(on_board yes)
 		(dnp no)
-		(property "Reference" "#PWR047"
+		(property "Reference" "#PWR045"
 			(at 137.16 60.96 0)
 			(effects
@@
 			(project "MX_IMU"
 				(path "/8ed38441-7d4e-4e89-870f-07e11c6dce38/39c93069-edc2-4035-8fc7-27a45736847d"
-					(reference "#PWR047")
+					(reference "#PWR045")
 					(unit 1)
 				)
@@
 			)
 		)
-		(property "Value" "16MHz"
+		(property "Value" "Crystal_GND24_Small"
 			(at 156.845 90.17 0)
 			(effects
@@
 			)
 		)
-		(property "Value" "47"
+		(property "Value" "R_Small"
 			(at 167.64 90.17 0)
 			(effects
@@
 			)
 		)
-		(property "Value" "12p"
+		(property "Value" "C_Small"
 			(at 168.91 102.87 0)
 			(effects
@@
 			)
 		)
-		(property "Value" "12p"
+		(property "Value" "C_Small"
 			(at 146.05 102.87 0)
 			(effects
@@
 			)
 		)
-		(property "Value" "10k"
+		(property "Value" "R_Small"
 			(at 180.34 149.86 0)
 			(effects
@@
 		(on_board yes)
 		(dnp no)
-		(property "Reference" "C26"
+		(property "Reference" "C21"
 			(at 241.5032 144.6784 0)
 			(effects
@@
 			)
 		)
-		(property "Value" "100nf"
+		(property "Value" "C_Small"
 			(at 241.5032 142.367 0)
 			(effects
@@
 			(project "MX_IMU"
 				(path "/8ed38441-7d4e-4e89-870f-07e11c6dce38/39c93069-edc2-4035-8fc7-27a45736847d"
-					(reference "C26")
+					(reference "C21")
 					(unit 1)
 				)
@@
 		(dnp no)
 		(fields_autoplaced yes)
-		(property "Reference" "D5"
+		(property "Reference" "D4"
 			(at 243.84 90.0998 0)
 			(effects
@@
 			(project ""
 				(path "/8ed38441-7d4e-4e89-870f-07e11c6dce38/39c93069-edc2-4035-8fc7-27a45736847d"
-					(reference "D5")
+					(reference "D4")
 					(unit 1)
 				)
@@
 		(dnp no)
 		(fields_autoplaced yes)
-		(property "Reference" "#PWR044"
+		(property "Reference" "#PWR048"
 			(at 229.87 90.17 0)
 			(effects
@@
 			(project "MX_IMU"
 				(path "/8ed38441-7d4e-4e89-870f-07e11c6dce38/39c93069-edc2-4035-8fc7-27a45736847d"
-					(reference "#PWR044")
+					(reference "#PWR048")
 					(unit 1)
 				)
@@
 		(on_board yes)
 		(dnp no)
-		(property "Reference" "#PWR049"
+		(property "Reference" "#PWR051"
 			(at 247.65 111.76 0)
 			(effects
@@
 			(project "MX_IMU"
 				(path "/8ed38441-7d4e-4e89-870f-07e11c6dce38/39c93069-edc2-4035-8fc7-27a45736847d"
-					(reference "#PWR049")
+					(reference "#PWR051")
 					(unit 1)
 				)
@@
 		(dnp no)
 		(fields_autoplaced yes)
-		(property "Reference" "#PWR048"
+		(property "Reference" "#PWR050"
 			(at 229.87 111.76 0)
 			(effects
@@
 			(project "MX_IMU"
 				(path "/8ed38441-7d4e-4e89-870f-07e11c6dce38/39c93069-edc2-4035-8fc7-27a45736847d"
-					(reference "#PWR048")
+					(reference "#PWR050")
 					(unit 1)
 				)
@@
 			)
 		)
-		(property "Value" "RESET"
+		(property "Value" "SW_Push"
 			(at 253.873 145.2122 90)
 			(effects
@@
 			)
 		)
-		(property "Value" "N_USB_VBUS"
+		(property "Value" "Jumper_2_Open"
 			(at 144.78 145.7761 0)
 			(effects
@@
 		(dnp no)
 		(fields_autoplaced yes)
-		(property "Reference" "#PWR065"
+		(property "Reference" "#PWR055"
 			(at 250.19 161.29 0)
 			(effects
@@
 			(project "MX_IMU"
 				(path "/8ed38441-7d4e-4e89-870f-07e11c6dce38/39c93069-edc2-4035-8fc7-27a45736847d"
-					(reference "#PWR065")
+					(reference "#PWR055")
 					(unit 1)
 				)
@@
 			)
 		)
-		(property "Value" "100nf"
+		(property "Value" "C_Small"
 			(at 249.9868 97.663 0)
 			(effects
@@
 		(dnp no)
 		(fields_autoplaced yes)
-		(property "Reference" "#PWR055"
+		(property "Reference" "#PWR056"
 			(at 154.94 162.56 0)
 			(effects
@@
 			(project "MX_IMU"
 				(path "/8ed38441-7d4e-4e89-870f-07e11c6dce38/39c93069-edc2-4035-8fc7-27a45736847d"
-					(reference "#PWR055")
+					(reference "#PWR056")
 					(unit 1)
 				)
@@
 			)
 		)
-		(property "Value" "10k"
+		(property "Value" "R"
 			(at 149.86 153.67 0)
 			(effects
@@
 		(dnp no)
 		(fields_autoplaced yes)
-		(property "Reference" "#PWR045"
+		(property "Reference" "#PWR049"
 			(at 247.65 90.17 0)
 			(effects
@@
 			(project "MX_IMU"
 				(path "/8ed38441-7d4e-4e89-870f-07e11c6dce38/39c93069-edc2-4035-8fc7-27a45736847d"
-					(reference "#PWR045")
+					(reference "#PWR049")
 					(unit 1)
 				)

Commit message: update
Parts:
- renumbered C22 to C11, C11 to C12, C23 to C13, C12 to C14, C13 to C15, C14 to C16, C15 to C17, C16 to C18, C17 to C19, C19 to C20, C20 to C21, C21 to C22, C18 to C23, R9 to R10, R10 to R11, R11 to R9

Commit message: update value for capacity and  resistor
Parts:
- C10: value C_Small -> 4u7
- C11, C13: value C_Small -> 2u2
- C12, C14, C15, C16, C17: value C_Small -> 100n
- C18: value C_Small -> 1u
- C19: value C_Small -> 10n
- C20, C21: value C_Small -> 12p
- C22, C23: value C_Small -> 100nf
- FB1: value FerriteBead_Small -> 600 @ 600 MHz
- R10: value R_Small -> 47
- R11: value R_Small -> 10k
- R9: value R -> 10k
- Y1: value Crystal_GND24_Small -> 16MHz
Other:
- note removed: "need replace LED with ws2812B"
Changed lines of the file:
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@@
 	(generator_version "9.0")
 	(paper "A4")
-	(text "need replace LED with ws2812B"
-		(exclude_from_sim no)
-		(at 246.888 77.47 0)
-		(effects
-			(font
-				(size 1.27 1.27)
-			)
-		)
-	)
 	(text "HSE"
 		(exclude_from_sim no)
@@
 			)
 		)
-		(property "Value" "C_Small"
+		(property "Value" "2u2"
 			(at 62.23 168.91 0)
 			(effects
@@
 			)
 		)
-		(property "Value" "C_Small"
+		(property "Value" "2u2"
 			(at 54.61 163.83 0)
 			(effects
@@
 			)
 		)
-		(property "Value" "C_Small"
+		(property "Value" "4u7"
 			(at 53.34 50.8 0)
 			(effects
@@
 			)
 		)
-		(property "Value" "C_Small"
+		(property "Value" "100n"
 			(at 62.23 50.8 0)
 			(effects
@@
 			)
 		)
-		(property "Value" "C_Small"
+		(property "Value" "100n"
 			(at 72.39 50.8 0)
 			(effects
@@
 			)
 		)
-		(property "Value" "C_Small"
+		(property "Value" "100n"
 			(at 82.55 50.8 0)
 			(effects
@@
 			)
 		)
-		(property "Value" "C_Small"
+		(property "Value" "100n"
 			(at 92.71 50.8 0)
 			(effects
@@
 			)
 		)
-		(property "Value" "C_Small"
+		(property "Value" "100n"
 			(at 102.87 50.8 0)
 			(effects
@@
 			)
 		)
-		(property "Value" "FerriteBead_Small"
+		(property "Value" "600 @ 600 MHz"
 			(at 127 50.165 90)
 			(effects
@@
 			)
 		)
-		(property "Value" "C_Small"
+		(property "Value" "1u"
 			(at 139.7 52.07 0)
 			(effects
@@
 			)
 		)
-		(property "Value" "C_Small"
+		(property "Value" "10n"
 			(at 151.13 52.07 0)
 			(effects
@@
 			)
 		)
-		(property "Value" "Crystal_GND24_Small"
-			(at 156.845 90.17 0)
+		(property "Value" "16MHz"
+			(at 175.514 95.25 0)
 			(effects
 				(font
@@
 			)
 		)
-		(property "Value" "R_Small"
+		(property "Value" "47"
 			(at 167.64 90.17 0)
 			(effects
@@
 			)
 		)
-		(property "Value" "C_Small"
+		(property "Value" "12p"
 			(at 168.91 102.87 0)
 			(effects
@@
 			)
 		)
-		(property "Value" "C_Small"
+		(property "Value" "12p"
 			(at 146.05 102.87 0)
 			(effects
@@
 			)
 		)
-		(property "Value" "R_Small"
+		(property "Value" "10k"
 			(at 180.34 149.86 0)
 			(effects
@@
 			)
 		)
-		(property "Value" "C_Small"
+		(property "Value" "100nf"
 			(at 241.5032 142.367 0)
 			(effects
@@
 			)
 		)
-		(property "Value" "C_Small"
+		(property "Value" "100nf"
 			(at 249.9868 97.663 0)
 			(effects
@@
 			)
 		)
-		(property "Value" "R"
+		(property "Value" "10k"
 			(at 149.86 153.67 0)
 			(effects

Commit message: update pcb and  imu 3d model
Changed lines of the file:
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@@
 		)
 		(property "Value" "16MHz"
-			(at 175.514 95.25 0)
+			(at 156.972 90.424 0)
 			(effects
 				(font

Commit message: save
Parts:
- removed C21: 12p, Capacitor_SMD:C_0402_1005Metric, symbol Device:C_Small
- removed R10: 47, Resistor_SMD:R_0402_1005Metric, symbol Device:R_Small
- removed Y1: 16MHz, Crystal:Crystal_SMD_3225-4Pin_3.2x2.5mm, symbol Device:Crystal_GND24_Small
- added U8: 8Mhz,50ppm, Oscillator:Oscillator_SMD_SeikoEpson_SG8002CE-4Pin_3.2x2.5mm, symbol bt_oscillator:OSC;12Mhz;50ppm;3v3;SG3225CAN
- C20: value 12p -> 100n; LCSC Part # C1547 -> C1525
- renumbered JP3 to BOOT1, C22 to C21, C23 to C22, D4 to MainLED1, R11 to R10, SW1 to Reset1
Connections:
- net +3.3V: now also C20.1, U8.1 (ST#), U8.4 (Vcc)
- net Flash_CS: now also U7.33 (PB12); no longer U7.37 (PC6)
- net GND: now also U8.2 (GND)
- net GYRO_CS: now also U7.26 (PB0); no longer U7.24 (PC4)
- net GYRO_INT1: now also U7.20 (PA4); no longer U7.26 (PB0)
- net HSE_IN: now also U8.3 (OUT); no longer C20.1
- net Status_LED: no longer U7.30 (PB11)
- net TELE_CTS: now reaches U7.14 (PA0)
- net TELE_RTS: now reaches U7.15 (PA1)
- net GYRO_INT2: now reaches U7.41 (PA8)
- net Serial_TX: now reaches U7.42 (PA9)
- net Serial_RX: now reaches U7.43 (PA10)
- net GPS_SCL: now reaches U7.61 (PB8)
- net GPS_SDA: now reaches U7.62 (PB9)
- net Flash_CLK renamed Flash_SCK
- net HSE_OUT: no longer names the net of U7.6 (PH1)
- net USART2_RX renamed TELE_RX
- net USART2_TX renamed TELE_TX
- net USART3_RX renamed GPS_RX
- net USART3_TX renamed GPS_TX
- no-connect marks 28 -> 23
