File: PowerSupply.kicad_sch (KiCad schematic)
At the start: 35 parts, among them J3 S2B-ZRLFSN, J5 Native USB, J6 Serial USB, U4 NCP1117-5.0_SOT223, U5 TPS2115ADRBR, U6 ld39150dt33-r, U7 USBLC6-2SC6, U8 USBLC6-2SC6, U9 CH340E

Commit message: update
Parts:
- renumbered C19 to C1, C22 to C2, C24 to C3, C23 to C4, C25 to C5, C20 to C6, C21 to C7, C26 to C8, C27 to C9, D3 to D1, D6 to D2, D7 to D3, J3 to J1, J5 to J2, J6 to J3, R15 to R1, R16 to R2, R14 to R3, R17 to R4, R18 to R5, R13 to R6, R21 to R7, R22 to R8, TP3 to TP2, TP2 to TP3, U7 to U1, U4 to U2, U6 to U3, U5 to U4, U8 to U5, U9 to U6

Commit message: update library
Parts:
- C1: value 10uf/30v -> C_Small
- C2, C5: value 10uf -> C_Small
- C3: value 2u2 -> C_Small
- C4: value 1u -> C
- C6, C7, C8, C9: value 100nf -> C_Small
- D1: value GREEN -> LED
- D2: value GREEN_TX -> LED
- D3: value RED_RX -> LED
- J1: footprint mylib:CONN_S2B-ZR_JST -> CONN_S2B-ZR_JST
- J3: value Serial USB -> Native USB
- JP1: value N_USB_VBUS -> Jumper_2_Open
- JP2: value S_USB_VBUS -> Jumper_2_Open
- R1, R2, R4, R5: value 5.1k -> R_Small
- R3: value R_LIM -> R_Small
- R6: value 10k -> R_Small
- R7: value 1k -> R_Small
- R8: value 2.2k -> R_Small
- TP1: value TP_REG_5V -> TestPoint
- TP2: value TP_VBUS_5V -> TestPoint
- TP3: value TP_3V3 -> TestPoint
- TP4: value TP_5V -> TestPoint
- U4: footprint mylib:SON65P300X300X100-9N -> 53-01:TPS2115ADRBR
Changed lines of the file:
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@@
 			)
 		)
-		(property "Value" "TP_REG_5V"
+		(property "Value" "TestPoint"
 			(at 20.32 78.74 0)
 			(effects
@@
 			)
 		)
-		(property "Value" "1u"
+		(property "Value" "C"
 			(at 105.41 60.96 0)
 			(effects
@@
 			)
 		)
-		(property "Value" "5.1k"
+		(property "Value" "R_Small"
 			(at 203.5658 43.8979 90)
 			(effects
@@
 			)
 		)
-		(property "Value" "TP_5V"
+		(property "Value" "TestPoint"
 			(at 35.56 100.33 0)
 			(effects
@@
 			)
 		)
-		(property "Value" "2u2"
+		(property "Value" "C_Small"
 			(at 130.81 59.69 0)
 			(effects
@@
 			)
 		)
-		(property "Value" "5.1k"
+		(property "Value" "R_Small"
 			(at 203.2 37.4705 90)
 			(effects
@@
 			)
 		)
-		(property "Value" "GREEN_TX"
+		(property "Value" "LED"
 			(at 64.77 156.21 0)
 			(effects
@@
 			)
 		)
-		(property "Value" "10uf/30v"
+		(property "Value" "C_Small"
 			(at 46.99 59.69 0)
 			(effects
@@
 			)
 		)
-		(property "Value" "10uf"
+		(property "Value" "C_Small"
 			(at 140.97 100.33 0)
 			(effects
@@
 			)
 		)
-		(property "Value" "TP_VBUS_5V"
+		(property "Value" "TestPoint"
 			(at 33.02 78.74 0)
 			(effects
@@
 			)
 		)
-		(property "Footprint" "mylib:CONN_S2B-ZR_JST"
+		(property "Footprint" "CONN_S2B-ZR_JST"
 			(at 36.83 39.37 0)
 			(effects
@@
 			)
 		)
-		(property "Value" "100nf"
+		(property "Value" "C_Small"
 			(at 58.42 104.14 0)
 			(effects
@@
 			)
 		)
-		(property "Value" "10k"
+		(property "Value" "R_Small"
 			(at 33.02 118.11 0)
 			(effects
@@
 			)
 		)
-		(property "Footprint" "mylib:SON65P300X300X100-9N"
+		(property "Footprint" "53-01:TPS2115ADRBR"
 			(at 107.95 84.074 0)
 			(effects
@@
 	)
 	(symbol
-		(lib_name "VCC_1")
 		(lib_id "power:VCC")
 		(at 66.04 85.09 0)
@@
 	)
 	(symbol
-		(lib_name "VCC_1")
 		(lib_id "power:VCC")
 		(at 57.15 49.53 0)
@@
 			)
 		)
-		(property "Value" "2.2k"
+		(property "Value" "R_Small"
 			(at 71.12 149.86 0)
 			(effects
@@
 			)
 		)
-		(property "Value" "GREEN"
+		(property "Value" "LED"
 			(at 38.1 123.19 0)
 			(effects
@@
 			)
 		)
-		(property "Value" "RED_RX"
+		(property "Value" "LED"
 			(at 73.66 156.21 0)
 			(effects
@@
 	)
 	(symbol
-		(lib_name "VCC_1")
 		(lib_id "power:VCC")
 		(at 36.83 36.83 0)
@@
 			)
 		)
-		(property "Value" "1k"
+		(property "Value" "R_Small"
 			(at 62.23 149.86 0)
 			(effects
@@
 			)
 		)
-		(property "Value" "S_USB_VBUS"
+		(property "Value" "Jumper_2_Open"
 			(at 220.98 81.0061 0)
 			(effects
@@
 	)
 	(symbol
-		(lib_name "VCC_1")
 		(lib_id "power:VCC")
 		(at 77.47 85.09 0)
@@
 			)
 		)
-		(property "Value" "5.1k"
+		(property "Value" "R_Small"
 			(at 203.5658 106.1279 90)
 			(effects
@@
 	)
 	(symbol
-		(lib_name "VCC_1")
 		(lib_id "power:VCC")
 		(at 25.4 68.58 0)
@@
 			)
 		)
-		(property "Value" "N_USB_VBUS"
+		(property "Value" "Jumper_2_Open"
 			(at 220.98 68.3061 0)
 			(effects
@@
 			)
 		)
-		(property "Value" "100nf"
+		(property "Value" "C_Small"
 			(at 69.85 104.14 0)
 			(effects
@@
 			)
 		)
-		(property "Value" "100nf"
+		(property "Value" "C_Small"
 			(at 82.55 149.86 0)
 			(effects
@@
 			)
 		)
-		(property "Value" "100nf"
+		(property "Value" "C_Small"
 			(at 29.21 148.59 0)
 			(effects
@@
 			)
 		)
-		(property "Value" "TP_3V3"
+		(property "Value" "TestPoint"
 			(at 21.59 100.33 0)
 			(effects
@@
 			)
 		)
-		(property "Value" "Serial USB"
+		(property "Value" "Native USB"
 			(at 166.37 92.71 0)
 			(effects
@@
 			)
 		)
-		(property "Value" "R_LIM"
+		(property "Value" "R_Small"
 			(at 83.82 88.2705 90)
 			(effects
@@
 			)
 		)
-		(property "Value" "5.1k"
+		(property "Value" "R_Small"
 			(at 203.2 99.7005 90)
 			(effects
@@
 			)
 		)
-		(property "Value" "10uf"
+		(property "Value" "C_Small"
 			(at 84.8741 60.1285 0)
 			(effects
@@
 	)
 	(symbol
-		(lib_name "VCC_1")
 		(lib_id "power:VCC")
 		(at 38.1 68.58 0)
@@
 	)
 	(symbol
-		(lib_name "VCC_1")
 		(lib_id "power:VCC")
 		(at 82.55 49.53 0)

Commit message: clean files
Parts:
- J1: footprint CONN_S2B-ZR_JST -> mylib:CONN_S2B-ZR_JST
- U4: footprint 53-01:TPS2115ADRBR -> mylib:SON65P300X300X100-9N
Changed lines of the file:
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@@
 			)
 		)
-		(property "Footprint" "CONN_S2B-ZR_JST"
+		(property "Footprint" "mylib:CONN_S2B-ZR_JST"
 			(at 36.83 39.37 0)
 			(effects
@@
 			)
 		)
-		(property "Footprint" "53-01:TPS2115ADRBR"
+		(property "Footprint" "mylib:SON65P300X300X100-9N"
 			(at 107.95 84.074 0)
 			(effects

Commit message: update
Parts:
- renumbered C8 to C1, C1 to C2, C6 to C3, C7 to C4, C9 to C5, C2 to C6, C4 to C7, C3 to C8, C5 to C9, R6 to R1, R7 to R2, R8 to R3, R3 to R4, R1 to R5, R2 to R6, R4 to R7, R5 to R8, TP3 to TP2, TP2 to TP3, U6 to U1, U4 to U3, U3 to U4, U1 to U5, U5 to U6

Commit message: update value for capacity and  resistor
Parts:
- C1, C3, C4, C5: value C_Small -> 100nf
- C2: value C_Small -> 10uf/30v
- C6, C9: value C_Small -> 10uf
- C7: value C -> 1u
- C8: value C_Small -> 2u2
- R1: value R_Small -> 330R
- R2, R3: value R_Small -> 330
- R4: value R_Small -> 390R
- R5, R6, R7, R8: value R_Small -> 5.1k
Changed lines of the file:
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@@
 			)
 		)
-		(property "Value" "C"
+		(property "Value" "1u"
 			(at 105.41 60.96 0)
 			(effects
@@
 			)
 		)
-		(property "Value" "R_Small"
+		(property "Value" "5.1k"
 			(at 203.5658 43.8979 90)
 			(effects
@@
 			)
 		)
-		(property "Value" "C_Small"
+		(property "Value" "2u2"
 			(at 130.81 59.69 0)
 			(effects
@@
 			)
 		)
-		(property "Value" "R_Small"
+		(property "Value" "5.1k"
 			(at 203.2 37.4705 90)
 			(effects
@@
 			)
 		)
-		(property "Value" "C_Small"
+		(property "Value" "10uf/30v"
 			(at 46.99 59.69 0)
 			(effects
@@
 			)
 		)
-		(property "Value" "C_Small"
+		(property "Value" "10uf"
 			(at 140.97 100.33 0)
 			(effects
@@
 			)
 		)
-		(property "Value" "C_Small"
+		(property "Value" "100nf"
 			(at 58.42 104.14 0)
 			(effects
@@
 			)
 		)
-		(property "Value" "R_Small"
+		(property "Value" "330R"
 			(at 33.02 118.11 0)
 			(effects
@@
 			)
 		)
-		(property "Value" "R_Small"
+		(property "Value" "330"
 			(at 71.12 149.86 0)
 			(effects
@@
 			)
 		)
-		(property "Value" "R_Small"
+		(property "Value" "330"
 			(at 62.23 149.86 0)
 			(effects
@@
 			)
 		)
-		(property "Value" "R_Small"
+		(property "Value" "5.1k"
 			(at 203.5658 106.1279 90)
 			(effects
@@
 			)
 		)
-		(property "Value" "C_Small"
+		(property "Value" "100nf"
 			(at 69.85 104.14 0)
 			(effects
@@
 			)
 		)
-		(property "Value" "C_Small"
+		(property "Value" "100nf"
 			(at 82.55 149.86 0)
 			(effects
@@
 			)
 		)
-		(property "Value" "C_Small"
+		(property "Value" "100nf"
 			(at 29.21 148.59 0)
 			(effects
@@
 			)
 		)
-		(property "Value" "R_Small"
+		(property "Value" "390R"
 			(at 83.82 88.2705 90)
 			(effects
@@
 			)
 		)
-		(property "Value" "R_Small"
+		(property "Value" "5.1k"
 			(at 203.2 99.7005 90)
 			(effects
@@
 		(fields_autoplaced yes)
 		(property "Reference" "C6"
-			(at 84.8741 57.5916 0)
+			(at 85.09 57.1562 0)
 			(effects
 				(font
@@
 			)
 		)
-		(property "Value" "C_Small"
-			(at 84.8741 60.1285 0)
+		(property "Value" "10uf"
+			(at 85.09 59.6962 0)
 			(effects
 				(font

Commit message: update
Connections:
- net USART3_RX renamed Serial_RX
- net USART3_TX renamed Serial_TX
Changed lines of the file:
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@@
+		)
+	)
+	(global_label "Serial_TX"
+		(shape input)
+		(at 86.36 162.56 0)
+		(effects
+			(font
+				(size 1.27 1.27)
+			)
+			(justify left)
+		)
+		(property "Intersheetrefs" "${INTERSHEET_REFS}"
+			(at 86.36 162.56 0)
+			(effects
+				(font
+					(size 1.27 1.27)
+				)
+				(hide yes)
+			)
 		)
 	)
@@
 		)
 	)
+	(global_label "Serial_RX"
+		(shape input)
+		(at 86.36 165.1 0)
+		(effects
+			(font
+				(size 1.27 1.27)
+			)
+			(justify left)
+		)
+		(property "Intersheetrefs" "${INTERSHEET_REFS}"
+			(at 86.36 165.1 0)
+			(effects
+				(font
+					(size 1.27 1.27)
+				)
+				(hide yes)
+			)
+		)
+	)
 	(global_label "C_Serial_D+"
 		(shape input)
@@
 		)
 	)
-	(global_label "USART3_TX"
-		(shape input)
-		(at 86.36 162.56 0)
-		(fields_autoplaced yes)
-		(effects
-			(font
-				(size 1.27 1.27)
-			)
-			(justify left)
-		)
-		(property "Intersheetrefs" "${INTERSHEET_REFS}"
-			(at 99.5656 162.56 0)
-			(effects
-				(font
-					(size 1.27 1.27)
-				)
-				(justify left)
-				(hide yes)
-			)
-		)
-	)
 	(global_label "Serial_D-"
 		(shape input)
@@
 			(effects
 				(font
-					(size 1.27 1.27)
-				)
-				(justify left)
-				(hide yes)
-			)
-		)
-	)
-	(global_label "USART3_RX"
-		(shape input)
-		(at 86.36 165.1 0)
-		(fields_autoplaced yes)
-		(effects
-			(font
-				(size 1.27 1.27)
-			)
-			(justify left)
-		)
-		(property "Intersheetrefs" "${INTERSHEET_REFS}"
-			(at 99.868 165.1 0)
-			(effects
-				(font

Commit message: update
Parts:
- removed JP1, JP2: Jumper_2_Open, Connector_PinHeader_2.54mm:PinHeader_1x02_P2.54mm_Vertical, symbol Jumper:Jumper_2_Open
- added SW2: SSSS213000, mylib:SSSS213000, symbol SSSS213000:SSSS213000
Connections:
- net Serial_VBUS is gone; now on net VBUS: C5.1, J3.A4 (VBUS), J3.A9 (VBUS), J3.B4 (VBUS), J3.B9 (VBUS), R2.1, R3.1, U1.7 (VCC), U6.5 (VBUS)
- net Native_VBUS: now also SW2.1 (NO)
- net VBUS: now also SW2.2 (C)
