File: PowerSupply.kicad_sch (KiCad schematic)
At the start: 35 parts, among them J1 S2B-ZRLFSN, J2 Native USB, J3 Native USB, U1 CH340E, U2 NCP1117-5.0_SOT223, U3 TPS2115ADRBR, U4 ld39150dt33-r, U5 USBLC6-2SC6, U6 USBLC6-2SC6

Commit message: update
Parts:
- removed JP1, JP2: Jumper_2_Open, Connector_PinHeader_2.54mm:PinHeader_1x02_P2.54mm_Vertical, symbol Jumper:Jumper_2_Open
- added SW2: SSSS213000, mylib:SSSS213000, symbol SSSS213000:SSSS213000
Connections:
- net Serial_VBUS is gone; now on net VBUS: C5.1, J3.A4 (VBUS), J3.A9 (VBUS), J3.B4 (VBUS), J3.B9 (VBUS), R2.1, R3.1, U1.7 (VCC), U6.5 (VBUS)
- net Native_VBUS: now also SW2.1 (NO)
- net VBUS: now also SW2.2 (C)

Commit message: update
Parts:
- removed J1: S2B-ZRLFSN, mylib:CONN_S2B-ZR_JST, symbol jst_zh:S2B-ZRLFSN
- added J1: B2B-PH-K-S, mylib:JST_B2B-PH-K-S, symbol B2B-PH-K-S:B2B-PH-K-S
- renumbered SW2 to SW1
Connections:
- net GND: now also J1.2
- net VBUS: no longer C5.1, J3.A4 (VBUS), J3.A9 (VBUS), J3.B4 (VBUS), J3.B9 (VBUS), R2.1, R3.1, U1.7 (VCC), U6.5 (VBUS)
- net VCC: now also J1.1
- net Serial_VBUS: now reaches SW1.3 (NC)
- net Serial_VBUS: now also C5.1, J3.A4 (VBUS), J3.A9 (VBUS), J3.B4 (VBUS), J3.B9 (VBUS), R2.1, R3.1, U1.7 (VCC), U6.5 (VBUS)

Commit message: update
Parts:
- SW1: footprint mylib:SSSS213000 -> SSSS213000
- renumbered C2 to C1, C6 to C2, C8 to C3, C7 to C4, C9 to C5, C3 to C6, C4 to C7, C1 to C8, C5 to C9, R5 to R1, R6 to R2, R4 to R3, R7 to R4, R8 to R5, R1 to R6, R2 to R7, R3 to R8, TP3 to TP2, TP2 to TP3, U5 to U1, U4 to U3, U3 to U4, U6 to U5, U1 to U6

Commit message: update
Parts:
- removed TP1, TP2, TP3, TP4: TestPoint, TestPoint:TestPoint_Pad_D1.0mm, symbol Connector:TestPoint

Commit message: update
Parts:
- SW1: footprint SSSS213000 -> mylib:SSSS213000
Changed lines of the file:
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@@
 	(wire
 		(pts
+			(xy 233.68 76.2) (xy 231.14 76.2)
+		)
+		(stroke
+			(width 0)
+			(type default)
+		)
+	)
+	(wire
+		(pts
 			(xy 241.3 110.49) (xy 240.03 110.49)
 		)
@@
 			)
 		)
-		(property "Footprint" "SSSS213000"
+		(property "Footprint" "mylib:SSSS213000"
 			(at 212.09 -18.72 0)
 			(effects
@@
 	(symbol
 		(lib_id "power:PWR_FLAG")
-		(at 231.14 76.2 270)
+		(at 233.68 76.2 270)
 		(unit 1)
 		(exclude_from_sim no)
@@
 		(fields_autoplaced yes)
 		(property "Reference" "#FLG04"
-			(at 233.045 76.2 0)
+			(at 235.585 76.2 0)
 			(effects
 				(font
@@
 		)
 		(property "Value" "PWR_FLAG"
-			(at 234.95 76.1999 90)
+			(at 237.49 76.1999 90)
 			(effects
 				(font
@@
 		)
 		(property "Footprint" ""
-			(at 231.14 76.2 0)
+			(at 233.68 76.2 0)
 			(effects
 				(font
@@
 		)
 		(property "Datasheet" "~"
-			(at 231.14 76.2 0)
+			(at 233.68 76.2 0)
 			(effects
 				(font
@@
 		)
 		(property "Description" "Special symbol for telling ERC where power comes from"
-			(at 231.14 76.2 0)
+			(at 233.68 76.2 0)
 			(effects
 				(font

Commit message: update
Parts:
- renumbered C8 to C1, C1 to C2, C6 to C3, C7 to C4, C9 to C5, C2 to C6, C4 to C7, C3 to C8, C5 to C9, R6 to R1, R7 to R2, R8 to R3, R3 to R4, R1 to R5, R2 to R6, R4 to R7, R5 to R8, U6 to U1, U4 to U3, U3 to U4, U1 to U5, U5 to U6

Commit message: update
Parts:
- SW1: LCSC Part #   (none) -> C125054
Changed lines of the file:
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@@
+			)
+		)
+		(property "LCSC Part #  " "C125054"
+			(at 231.14 76.2 0)
+			(effects
+				(font
+					(size 1.27 1.27)
+				)
+				(hide yes)
 			)
 		)
