File: Periph.kicad_sch (KiCad schematic)
At the start: 11 parts, among them U10 ICM-42688-P, U9 W25Q128JVS

Commit message: update
Parts:
- added C24, C25: 100n, Capacitor_SMD:C_0201_0603Metric, symbol Device:C_Small
- added R11, R12: 4.7k, Resistor_SMD:R_0603_1608Metric, symbol Device:R_Small
- added U9: BMP388, mylib:BMP388, symbol BMP388:BMP388
- renumbered C25 to C26, C26 to C27, C27 to C28, C24 to C29, R11 to R14, R12 to R15, U9 to U11
Connections:
- net +3.3V: now also C24.2, C25.1, R11.2, R12.2, U9.1 (VDDIO), U9.10 (VDD), U9.6 (CSB)
- net GND: now also C24.1, C25.2, U9.3 (VSS), U9.5 (SDO), U9.8 (VSS__1), U9.9 (VSS__2)
- new net BARO_INT: U9.7 (INT)
- new net Baro_SCL: R11.1, U9.2 (SCK)
- new net Baro_SDA: R12.1, U9.4 (SDI)
Other:
- note added: "Barometer"
- note added: "I2C Pullup"
- moved on the sheet: C23, C26, C27, C28, C29, LSE1, R13, R14, R15, U10, U11

Commit message: update
Parts:
- added J4: SM03B-GHS-TBLFSN, mylib:CONN_SM03B-GHS-TBLFSN_JST, symbol SM03B-GHS:SM03B-GHS-TBLFSN
- renumbered C29 to C24, C26 to C25, C27 to C26, C28 to C27, C24 to C28, C25 to C29, R14 to R11, R15 to R12, R11 to R14, R12 to R15, U9 to U11, U11 to U9
Connections:
- net Baro_SCL: now also J4.2
- net Baro_SDA: now also J4.1
- net GND: now also J4.3, J4.4, J4.5

Commit message: PumbaaV2_RC2
Parts:
- removed J4: SM03B-GHS-TBLFSN, mylib:CONN_SM03B-GHS-TBLFSN_JST, symbol SM03B-GHS:SM03B-GHS-TBLFSN
- added J4: SM04B-GHS-TB(LF)(SN), mylib:CONN_SM04B-GHS-TB_JST, symbol SM04B-GHS-TB:SM04B-GHS-TB
- C28, C29: footprint Capacitor_SMD:C_0201_0603Metric -> Capacitor_SMD:C_0402_1005Metric; LCSC Part # (none) -> C1525
- LSE1: LCSC Part  (none) -> C2650753 C5280579
- U11: LCSC Part (none) -> # C779278
- U9: value W25Q128JVS -> W25Q128JVSIQ; LCSC Part  (none) -> C97521
Connections:
- net +3.3V: now also J4.1
- net Baro_SCL: now also J4.4
- net Baro_SDA: now also J4.3
- net GND: now also J4.2, J4.5, J4.6
- net BARO_INT renamed Baro_INT
Other:
- moved on the sheet: C23, C24, C25, C26, C27, LSE1, R11, R12, R13, R14, R15, U11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
