File: Periph.kicad_sch (KiCad schematic)
At the start: 17 parts, among them J4 SM03B-GHS-TBLFSN, U10 ICM-42688-P, U11 BMP388, U9 W25Q128JVS

Commit message: update
Parts:
- LSE1: LCSC Part  (none) -> C2650753
Connections:
- net BARO_INT renamed Baro_INT
Changed lines of the file:
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@@
 		)
 	)
-	(global_label "BARO_INT"
+	(global_label "Baro_INT"
 		(shape input)
 		(at 214.63 59.69 0)
@@
 		)
 		(property "Intersheetrefs" "${INTERSHEET_REFS}"
-			(at 225.8726 59.6106 0)
+			(at 225.8399 59.69 0)
 			(effects
 				(font
@@
 			)
 		)
-		(property "Datasheet" ""
+		(property "Datasheet" "https://www.lcsc.com/datasheet/C2650753.pdf"
 			(at 82.55 38.1 0)
 			(effects
@@
 			)
 		)
-		(property "Description" ""
+		(property "Description" "3.3V 3.5mA CMOS SMD3225-4P Crystals RoHS 25ppm"
 			(at 82.55 38.1 0)
 			(effects
@@
 				(hide yes)
 			)
+		)
+		(property "LCSC Part " "C2650753"
+			(at 82.55 38.1 0)
+			(effects
+				(font
+					(size 1.27 1.27)
+				)
+				(hide yes)
+			)

Commit message: update spi flash
Parts:
- U9: value W25Q128JVS -> W25Q128JVSIQ; LCSC Part  (none) -> C97521
Changed lines of the file:
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@@
 			)
 		)
-		(property "Value" "W25Q128JVS"
+		(property "Value" "W25Q128JVSIQ"
 			(at 63.5 156.2099 0)
 			(effects
@@
 			(effects
 				(font
+					(size 1.27 1.27)
+				)
+				(hide yes)
+			)
+		)
+		(property "LCSC Part " "C97521"
+			(at 52.07 154.94 0)
+			(effects
+				(font

Commit message: update
Parts:
- U11: LCSC Part (none) -> # C779278
Changed lines of the file:
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@@
 			)
 		)
-		(property "Datasheet" ""
+		(property "Datasheet" "https://www.lcsc.com/datasheet/C779278.pdf"
 			(at 201.93 64.77 0)
 			(effects
@@
 			)
 		)
-		(property "Description" ""
+		(property "Description" "30Kpa~1.25bar LGA-10(2x2) Pressure Sensors, Transducers RoHS"
 			(at 201.93 64.77 0)
 			(effects
@@
 				(hide yes)
 			)
+		)
+		(property "LCSC Part" " #  C779278 "
+			(at 201.93 64.77 0)
+			(effects
+				(font
+					(size 1.27 1.27)
+				)
+				(hide yes)
+			)

Commit message: update
Parts:
- removed J4: SM03B-GHS-TBLFSN, mylib:CONN_SM03B-GHS-TBLFSN_JST, symbol SM03B-GHS:SM03B-GHS-TBLFSN
- added J4: SM04B-GHS-TB, mylib:CONN_SM04B-GHS-TB_JST, symbol SM04B-GHS-TB:SM04B-GHS-TB
Connections:
- net +3.3V: now also J4.1
- net Baro_SCL: now also J4.4
- net Baro_SDA: now also J4.3
- net GND: now also J4.2, J4.5, J4.6
Changed lines of the file:
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@@
 	)
 	(junction
-		(at 213.36 96.52)
+		(at 229.87 46.99)
 		(diameter 0)
 		(color 0 0 0 0)
 	)
 	(junction
-		(at 229.87 46.99)
+		(at 186.69 67.31)
 		(diameter 0)
 		(color 0 0 0 0)
 	)
 	(junction
-		(at 186.69 67.31)
+		(at 86.36 99.06)
 		(diameter 0)
 		(color 0 0 0 0)
 	)
 	(junction
-		(at 86.36 99.06)
+		(at 213.36 92.71)
 		(diameter 0)
 		(color 0 0 0 0)
@@
 	(wire
 		(pts
+			(xy 195.58 86.36) (xy 193.04 86.36)
+		)
+		(stroke
+			(width 0)
+			(type default)
+		)
+	)
+	(wire
+		(pts
 			(xy 214.63 52.07) (xy 222.25 52.07)
 		)
@@
 	(wire
 		(pts
+			(xy 170.18 93.98) (xy 195.58 93.98)
+		)
+		(stroke
+			(width 0)
+			(type default)
+		)
+	)
+	(wire
+		(pts
 			(xy 36.83 165.1) (xy 36.83 157.48)
 		)
@@
 	(wire
 		(pts
-			(xy 213.36 91.44) (xy 213.36 96.52)
-		)
-		(stroke
-			(width 0)
-			(type default)
-		)
-	)
-	(wire
-		(pts
 			(xy 135.89 74.93) (xy 135.89 77.47)
 		)
@@
 	(wire
 		(pts
+			(xy 213.36 88.9) (xy 213.36 92.71)
+		)
+		(stroke
+			(width 0)
+			(type default)
+		)
+	)
+	(wire
+		(pts
 			(xy 241.3 46.99) (xy 240.03 46.99)
 		)
@@
 	(wire
 		(pts
+			(xy 213.36 92.71) (xy 213.36 97.79)
+		)
+		(stroke
+			(width 0)
+			(type default)
+		)
+	)
+	(wire
+		(pts
 			(xy 127 68.58) (xy 135.89 68.58)
 		)
@@
 		)
 	)
+	(wire
+		(pts
+			(xy 195.58 88.9) (xy 193.04 88.9)
+		)
+		(stroke
+			(width 0)
+			(type default)
+		)
+	)
 	(polyline
 		(pts
@@
 	(wire
 		(pts
-			(xy 195.58 93.98) (xy 170.18 93.98)
-		)
-		(stroke
-			(width 0)
-			(type default)
-		)
-	)
-	(wire
-		(pts
 			(xy 83.82 71.12) (xy 87.63 71.12)
 		)
@@
 	(symbol
 		(lib_id "power:GND")
-		(at 195.58 96.52 0)
+		(at 193.04 88.9 270)
 		(unit 1)
 		(exclude_from_sim no)
@@
 		(fields_autoplaced yes)
 		(property "Reference" "#PWR074"
-			(at 195.58 102.87 0)
+			(at 186.69 88.9 0)
 			(effects
 				(font
@@
 		)
 		(property "Value" "GND"
-			(at 195.58 101.6 0)
+			(at 187.96 88.9 0)
 			(effects
 				(font
@@
 		)
 		(property "Footprint" ""
-			(at 195.58 96.52 0)
+			(at 193.04 88.9 0)
 			(effects
 				(font
@@
 		)
 		(property "Datasheet" ""
-			(at 195.58 96.52 0)
+			(at 193.04 88.9 0)
 			(effects
 				(font
@@
 		)
 		(property "Description" ""
-			(at 195.58 96.52 0)
+			(at 193.04 88.9 0)
 			(effects
 				(font
@@
 	)
 	(symbol
-		(lib_id "SM03B-GHS:SM03B-GHS-TBLFSN")
-		(at 195.58 91.44 0)
+		(lib_id "power:GND")
+		(at 81.28 166.37 0)
 		(unit 1)
 		(exclude_from_sim no)
@@
 		(on_board yes)
 		(dnp no)
-		(property "Reference" "J4"
-			(at 212.852 94.742 0)
+		(property "Reference" "#PWR066"
+			(at 81.28 172.72 0)
 			(effects
 				(font
-					(size 1.524 1.524)
+					(size 1.27 1.27)
 				)
-				(justify left)
+				(hide yes)
 			)
 		)
-		(property "Value" "SM03B-GHS-TBLFSN"
-			(at 209.55 95.2499 0)
+		(property "Value" "GND"
+			(at 81.407 170.7642 0)
 			(effects
 				(font
-					(size 1.524 1.524)
+					(size 1.27 1.27)
 				)
-				(justify left)
-				(hide yes)
 			)
 		)
-		(property "Footprint" "mylib:CONN_SM03B-GHS-TBLFSN_JST"
-			(at 195.58 91.44 0)
+		(property "Footprint" ""
+			(at 81.28 166.37 0)
 			(effects
 				(font
 					(size 1.27 1.27)
-					(italic yes)
 				)
 				(hide yes)
 			)
 		)
-		(property "Datasheet" "SM03B-GHS-TBLFSN"
-			(at 195.58 91.44 0)
+		(property "Datasheet" ""
+			(at 81.28 166.37 0)
 			(effects
 				(font
 					(size 1.27 1.27)
-					(italic yes)
 				)
 				(hide yes)
@@
 		)
 		(property "Description" ""
-			(at 195.58 91.44 0)
+			(at 81.28 166.37 0)
 			(effects
 				(font
 					(size 1.27 1.27)
 				)
-				(hide yes)
 			)
 		)
-		(pin "3"
-		)
-		(pin "2"
-		)
 		(pin "1"
 		)
-		(pin "5"
-		)
-		(pin "4"
-		)
 		(instances
-			(project ""
+			(project "MX_IMU"
 				(path "/8ed38441-7d4e-4e89-870f-07e11c6dce38/57f4b5bf-da86-4b65-9b05-7c9ef99c472c"
-					(reference "J4")
+					(reference "#PWR066")
 					(unit 1)
 				)
@@
 	)
 	(symbol
-		(lib_id "power:GND")
-		(at 81.28 166.37 0)
+		(lib_id "SM04B-GHS-TB:SM04B-GHS-TB")
+		(at 195.58 86.36 0)
 		(unit 1)
 		(exclude_from_sim no)
@@
 		(on_board yes)
 		(dnp no)
-		(property "Reference" "#PWR066"
-			(at 81.28 172.72 0)
+		(property "Reference" "J4"
+			(at 200.914 81.28 0)
 			(effects
 				(font
-					(size 1.27 1.27)
+					(size 1.524 1.524)
 				)
-				(hide yes)
+				(justify left)
 			)
 		)
-		(property "Value" "GND"
-			(at 81.407 170.7642 0)
+		(property "Value" "SM04B-GHS-TB"
+			(at 209.55 91.4399 0)
 			(effects
 				(font
-					(size 1.27 1.27)
+					(size 1.524 1.524)
 				)
+				(justify left)
+				(hide yes)
 			)
 		)
-		(property "Footprint" ""
-			(at 81.28 166.37 0)
+		(property "Footprint" "mylib:CONN_SM04B-GHS-TB_JST"
+			(at 195.58 86.36 0)
 			(effects
 				(font
 					(size 1.27 1.27)
+					(italic yes)
 				)
 				(hide yes)
 			)
 		)
-		(property "Datasheet" ""
-			(at 81.28 166.37 0)
+		(property "Datasheet" "SM04B-GHS-TB"
+			(at 195.58 86.36 0)
 			(effects
 				(font
 					(size 1.27 1.27)
+					(italic yes)
 				)
 				(hide yes)
@@
 		)
 		(property "Description" ""
-			(at 81.28 166.37 0)
+			(at 195.58 86.36 0)
 			(effects
 				(font
 					(size 1.27 1.27)
 				)
+				(hide yes)
 			)
 		)
+		(pin "4"
+		)
+		(pin "3"
+		)
+		(pin "2"
+		)
 		(pin "1"
 		)
+		(pin "5"
+		)
+		(pin "6"
+		)
 		(instances
 			(project "MX_IMU"
 				(path "/8ed38441-7d4e-4e89-870f-07e11c6dce38/57f4b5bf-da86-4b65-9b05-7c9ef99c472c"
-					(reference "#PWR066")
+					(reference "J4")
 					(unit 1)
 				)
@@
 	)
 	(symbol
+		(lib_id "power:+3.3V")
+		(at 193.04 86.36 0)
+		(unit 1)
+		(exclude_from_sim no)
+		(in_bom yes)
+		(on_board yes)
+		(dnp no)
+		(property "Reference" "#PWR0100"
+			(at 193.04 90.17 0)
+			(effects
+				(font
+					(size 1.27 1.27)
+				)
+				(hide yes)
+			)
+		)
+		(property "Value" "+3.3V"
+			(at 189.992 83.058 0)
+			(effects
+				(font
+					(size 1.27 1.27)
+				)
+			)
+		)
+		(property "Footprint" ""
+			(at 193.04 86.36 0)
+			(effects
+				(font
+					(size 1.27 1.27)
+				)
+				(hide yes)
+			)
+		)
+		(property "Datasheet" ""
+			(at 193.04 86.36 0)
+			(effects
+				(font
+					(size 1.27 1.27)
+				)
+				(hide yes)
+			)
+		)
+		(property "Description" ""
+			(at 193.04 86.36 0)
+			(effects
+				(font
+					(size 1.27 1.27)
+				)
+			)
+		)
+		(pin "1"
+		)
+		(instances
+			(project "MX_IMU"
+				(path "/8ed38441-7d4e-4e89-870f-07e11c6dce38/57f4b5bf-da86-4b65-9b05-7c9ef99c472c"
+					(reference "#PWR0100")
+					(unit 1)
+				)
+			)
+		)
+	)
+	(symbol
 		(lib_id "ASEK-32.768KHZ-L-R-T:ASEK-32.768KHZ-L-R-T")
 		(at 82.55 38.1 180)
@@
 	(symbol
 		(lib_id "power:GND")
-		(at 213.36 96.52 0)
+		(at 213.36 97.79 0)
 		(unit 1)
 		(exclude_from_sim no)
@@
 		(fields_autoplaced yes)
 		(property "Reference" "#PWR099"
-			(at 213.36 102.87 0)
+			(at 213.36 104.14 0)
 			(effects
 				(font
@@
 		)
 		(property "Value" "GND"
-			(at 213.36 101.6 0)
+			(at 213.36 102.87 0)
 			(effects
 				(font
@@
 		)
 		(property "Footprint" ""
-			(at 213.36 96.52 0)
+			(at 213.36 97.79 0)
 			(effects
 				(font
@@
 		)
 		(property "Datasheet" ""
-			(at 213.36 96.52 0)
+			(at 213.36 97.79 0)
 			(effects
 				(font
@@
 		)
 		(property "Description" ""
-			(at 213.36 96.52 0)
+			(at 213.36 97.79 0)
 			(effects
 				(font

Commit message: update for production
Changed lines of the file:
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@@
 		(dnp no)
 		(fields_autoplaced yes)
-		(property "Reference" "#PWR074"
+		(property "Reference" "#PWR078"
 			(at 186.69 88.9 0)
 			(effects
@@
 			(project "MX_IMU"
 				(path "/8ed38441-7d4e-4e89-870f-07e11c6dce38/57f4b5bf-da86-4b65-9b05-7c9ef99c472c"
-					(reference "#PWR074")
+					(reference "#PWR078")
 					(unit 1)
 				)
@@
 		(dnp no)
 		(fields_autoplaced yes)
-		(property "Reference" "#PWR076"
+		(property "Reference" "#PWR081"
 			(at 224.79 74.93 0)
 			(effects
@@
 			(project "MX_IMU"
 				(path "/8ed38441-7d4e-4e89-870f-07e11c6dce38/57f4b5bf-da86-4b65-9b05-7c9ef99c472c"
-					(reference "#PWR076")
+					(reference "#PWR081")
 					(unit 1)
 				)
@@
 		(on_board yes)
 		(dnp no)
-		(property "Reference" "#PWR059"
+		(property "Reference" "#PWR062"
 			(at 36.83 157.48 0)
 			(effects
@@
 			(project "MX_IMU"
 				(path "/8ed38441-7d4e-4e89-870f-07e11c6dce38/57f4b5bf-da86-4b65-9b05-7c9ef99c472c"
-					(reference "#PWR059")
+					(reference "#PWR062")
 					(unit 1)
 				)
@@
 		(dnp no)
 		(fields_autoplaced yes)
-		(property "Reference" "#PWR070"
+		(property "Reference" "#PWR073"
 			(at 116.84 69.85 0)
 			(effects
@@
 			(project "MX_IMU"
 				(path "/8ed38441-7d4e-4e89-870f-07e11c6dce38/57f4b5bf-da86-4b65-9b05-7c9ef99c472c"
-					(reference "#PWR070")
+					(reference "#PWR073")
 					(unit 1)
 				)
@@
 		(dnp no)
 		(fields_autoplaced yes)
-		(property "Reference" "#PWR063"
+		(property "Reference" "#PWR066"
 			(at 62.23 26.67 0)
 			(effects
@@
 			(project "MX_IMU"
 				(path "/8ed38441-7d4e-4e89-870f-07e11c6dce38/57f4b5bf-da86-4b65-9b05-7c9ef99c472c"
-					(reference "#PWR063")
+					(reference "#PWR066")
 					(unit 1)
 				)
@@
 		(dnp no)
 		(fields_autoplaced yes)
-		(property "Reference" "#PWR065"
+		(property "Reference" "#PWR068"
 			(at 81.28 144.78 0)
 			(effects
@@
 			(project ""
 				(path "/8ed38441-7d4e-4e89-870f-07e11c6dce38/57f4b5bf-da86-4b65-9b05-7c9ef99c472c"
-					(reference "#PWR065")
+					(reference "#PWR068")
 					(unit 1)
 				)
@@
 		(dnp no)
 		(fields_autoplaced yes)
-		(property "Reference" "#PWR067"
+		(property "Reference" "#PWR070"
 			(at 86.36 107.95 0)
 			(effects
@@
 			(project "MX_IMU"
 				(path "/8ed38441-7d4e-4e89-870f-07e11c6dce38/57f4b5bf-da86-4b65-9b05-7c9ef99c472c"
-					(reference "#PWR067")
+					(reference "#PWR070")
 					(unit 1)
 				)
@@
 		(dnp no)
 		(fields_autoplaced yes)
-		(property "Reference" "#PWR077"
+		(property "Reference" "#PWR082"
 			(at 222.25 48.26 0)
 			(effects
@@
 			(project "MX_IMU"
 				(path "/8ed38441-7d4e-4e89-870f-07e11c6dce38/57f4b5bf-da86-4b65-9b05-7c9ef99c472c"
-					(reference "#PWR077")
+					(reference "#PWR082")
 					(unit 1)
 				)
@@
 		(on_board yes)
 		(dnp no)
-		(property "Reference" "#PWR066"
+		(property "Reference" "#PWR069"
 			(at 81.28 172.72 0)
 			(effects
@@
 			(project "MX_IMU"
 				(path "/8ed38441-7d4e-4e89-870f-07e11c6dce38/57f4b5bf-da86-4b65-9b05-7c9ef99c472c"
-					(reference "#PWR066")
+					(reference "#PWR069")
 					(unit 1)
 				)
@@
 		(dnp no)
 		(fields_autoplaced yes)
-		(property "Reference" "#PWR078"
+		(property "Reference" "#PWR083"
 			(at 229.87 49.53 0)
 			(effects
@@
 			(project "MX_IMU"
 				(path "/8ed38441-7d4e-4e89-870f-07e11c6dce38/57f4b5bf-da86-4b65-9b05-7c9ef99c472c"
-					(reference "#PWR078")
+					(reference "#PWR083")
 					(unit 1)
 				)
@@
 		(dnp no)
 		(fields_autoplaced yes)
-		(property "Reference" "#PWR060"
+		(property "Reference" "#PWR063"
 			(at 49.53 54.61 0)
 			(effects
@@
 			(project "MX_IMU"
 				(path "/8ed38441-7d4e-4e89-870f-07e11c6dce38/57f4b5bf-da86-4b65-9b05-7c9ef99c472c"
-					(reference "#PWR060")
+					(reference "#PWR063")
 					(unit 1)
 				)
@@
 		(dnp no)
 		(fields_autoplaced yes)
-		(property "Reference" "#PWR079"
+		(property "Reference" "#PWR084"
 			(at 241.3 39.37 0)
 			(effects
@@
 			(project "MX_IMU"
 				(path "/8ed38441-7d4e-4e89-870f-07e11c6dce38/57f4b5bf-da86-4b65-9b05-7c9ef99c472c"
-					(reference "#PWR079")
+					(reference "#PWR084")
 					(unit 1)
 				)
@@
 		(dnp no)
 		(fields_autoplaced yes)
-		(property "Reference" "#PWR080"
+		(property "Reference" "#PWR085"
 			(at 248.92 50.8 0)
 			(effects
@@
 			(project "MX_IMU"
 				(path "/8ed38441-7d4e-4e89-870f-07e11c6dce38/57f4b5bf-da86-4b65-9b05-7c9ef99c472c"
-					(reference "#PWR080")
+					(reference "#PWR085")
 					(unit 1)
 				)
@@
 		(dnp no)
 		(fields_autoplaced yes)
-		(property "Reference" "#PWR073"
+		(property "Reference" "#PWR076"
 			(at 189.23 81.28 0)
 			(effects
@@
 			(project "MX_IMU"
 				(path "/8ed38441-7d4e-4e89-870f-07e11c6dce38/57f4b5bf-da86-4b65-9b05-7c9ef99c472c"
-					(reference "#PWR073")
+					(reference "#PWR076")
 					(unit 1)
 				)
@@
 		(dnp no)
 		(fields_autoplaced yes)
-		(property "Reference" "#PWR071"
+		(property "Reference" "#PWR074"
 			(at 135.89 85.09 0)
 			(effects
@@
 			(project "MX_IMU"
 				(path "/8ed38441-7d4e-4e89-870f-07e11c6dce38/57f4b5bf-da86-4b65-9b05-7c9ef99c472c"
-					(reference "#PWR071")
+					(reference "#PWR074")
 					(unit 1)
 				)
@@
 		(dnp no)
 		(fields_autoplaced yes)
-		(property "Reference" "#PWR072"
+		(property "Reference" "#PWR075"
 			(at 186.69 57.15 0)
 			(effects
@@
 			(project "MX_IMU"
 				(path "/8ed38441-7d4e-4e89-870f-07e11c6dce38/57f4b5bf-da86-4b65-9b05-7c9ef99c472c"
-					(reference "#PWR072")
+					(reference "#PWR075")
 					(unit 1)
 				)
@@
 		(dnp no)
 		(fields_autoplaced yes)
-		(property "Reference" "#PWR062"
+		(property "Reference" "#PWR065"
 			(at 52.07 173.99 0)
 			(effects
@@
 			(project "MX_IMU"
 				(path "/8ed38441-7d4e-4e89-870f-07e11c6dce38/57f4b5bf-da86-4b65-9b05-7c9ef99c472c"
-					(reference "#PWR062")
+					(reference "#PWR065")
 					(unit 1)
 				)
@@
 		(on_board yes)
 		(dnp no)
-		(property "Reference" "#PWR0100"
+		(property "Reference" "#PWR077"
 			(at 193.04 90.17 0)
 			(effects
@@
 			(project "MX_IMU"
 				(path "/8ed38441-7d4e-4e89-870f-07e11c6dce38/57f4b5bf-da86-4b65-9b05-7c9ef99c472c"
-					(reference "#PWR0100")
+					(reference "#PWR077")
 					(unit 1)
 				)
@@
 		(dnp no)
 		(fields_autoplaced yes)
-		(property "Reference" "#PWR069"
+		(property "Reference" "#PWR072"
 			(at 107.95 149.86 0)
 			(effects
@@
 			(project ""
 				(path "/8ed38441-7d4e-4e89-870f-07e11c6dce38/57f4b5bf-da86-4b65-9b05-7c9ef99c472c"
-					(reference "#PWR069")
+					(reference "#PWR072")
 					(unit 1)
 				)
@@
 		(dnp no)
 		(fields_autoplaced yes)
-		(property "Reference" "#PWR075"
+		(property "Reference" "#PWR079"
 			(at 213.36 36.83 0)
 			(effects
@@
 			(project "MX_IMU"
 				(path "/8ed38441-7d4e-4e89-870f-07e11c6dce38/57f4b5bf-da86-4b65-9b05-7c9ef99c472c"
-					(reference "#PWR075")
+					(reference "#PWR079")
 					(unit 1)
 				)
@@
 		(dnp no)
 		(fields_autoplaced yes)
-		(property "Reference" "#PWR068"
+		(property "Reference" "#PWR071"
 			(at 87.63 69.85 0)
 			(effects
@@
 			(project "MX_IMU"
 				(path "/8ed38441-7d4e-4e89-870f-07e11c6dce38/57f4b5bf-da86-4b65-9b05-7c9ef99c472c"
-					(reference "#PWR068")
+					(reference "#PWR071")
 					(unit 1)
 				)
@@
 					(size 1.27 1.27)
 				)
+				(hide yes)
 			)
 		)
@@
 					(size 1.27 1.27)
 				)
+				(hide yes)
 			)
 		)
@@
 		(dnp no)
 		(fields_autoplaced yes)
-		(property "Reference" "#PWR099"
+		(property "Reference" "#PWR080"
 			(at 213.36 104.14 0)
 			(effects
@@
 			(project "MX_IMU"
 				(path "/8ed38441-7d4e-4e89-870f-07e11c6dce38/57f4b5bf-da86-4b65-9b05-7c9ef99c472c"
-					(reference "#PWR099")
+					(reference "#PWR080")
 					(unit 1)
 				)
@@
 		(dnp no)
 		(fields_autoplaced yes)
-		(property "Reference" "#PWR081"
+		(property "Reference" "#PWR086"
 			(at 259.08 50.8 0)
 			(effects
@@
 			(project "MX_IMU"
 				(path "/8ed38441-7d4e-4e89-870f-07e11c6dce38/57f4b5bf-da86-4b65-9b05-7c9ef99c472c"
-					(reference "#PWR081")
+					(reference "#PWR086")
 					(unit 1)
 				)
@@
 		(dnp no)
 		(fields_autoplaced yes)
-		(property "Reference" "#PWR064"
+		(property "Reference" "#PWR067"
 			(at 62.23 39.37 0)
 			(effects
@@
 			(project "MX_IMU"
 				(path "/8ed38441-7d4e-4e89-870f-07e11c6dce38/57f4b5bf-da86-4b65-9b05-7c9ef99c472c"
-					(reference "#PWR064")
+					(reference "#PWR067")
 					(unit 1)
 				)
@@
 		(dnp no)
 		(fields_autoplaced yes)
-		(property "Reference" "#PWR061"
+		(property "Reference" "#PWR064"
 			(at 52.07 146.05 0)
 			(effects
@@
 			(project "MX_IMU"
 				(path "/8ed38441-7d4e-4e89-870f-07e11c6dce38/57f4b5bf-da86-4b65-9b05-7c9ef99c472c"
-					(reference "#PWR061")
-					(unit 1)
-				)
+					(reference "#PWR064")
+					(unit 1)
+				)
