File: MX_IMU.kicad_pcb (KiCad board)
At the start: 4 copper layers, 50 x 80 mm, 85 parts, among them J1 B2B-PH-K-S, J2 Native USB, J3 Native USB, J4 SM03B-GHS-TBLFSN, J5 Conn_02x03_Odd_Even, J6 Conn_02x03_Odd_Even, SW1 SSSS213000, SW2 SSSS213000, U1 CH340E, U10 ICM-42688-P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

Commit message: update
Other:
- board text added: "TELE"
Changed lines of the file:
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@@
 		(layer "Edge.Cuts")
+	)
+	(gr_text "TELE"
+		(at 162.708812 76.694083 0)
+		(layer "F.SilkS")
+		(effects
+			(font
+				(size 0.6 0.6)
+				(thickness 0.15)
+			)
+			(justify left bottom)
+		)
 	)
 	(gr_text "PC9\n"

Commit message: update
Parts:
- moved C8 1.00 mm to (139.0, 62.1)
- moved D1 1.00 mm to (141.3, 64.5)
- moved R1 1.00 mm to (138.3, 64.5)
- moved U4 1.00 mm to (142.8, 57.3)
Routing:
- net GND: track 164.3 -> 169.4 mm, vias 72 -> 75
- net +3.3V: track 62.6 -> 64.4 mm, vias 23 -> 24
- net Net-(U9-~{HOLD}/~{RESET}/IO_{3}): track 4.41 -> 3.60 mm

Commit message: update
Routing:
- net +3.3V: track 64.4 -> 67.6 mm, vias 24 -> 26
- net GND: track 169.4 -> 170.6 mm, vias 75 -> 76
- net Tim8_4: track 32.6 -> 33.4 mm
- net Tim8_2: track 28.1 -> 28.7 mm
- net Tim8_3: track 30.4 -> 30.9 mm

Commit message: update
Routing:
- net GND: track 170.6 -> 169.5 mm, vias 76 -> 77
- net +3.3V: track 67.6 -> 68.5 mm, vias 26 -> 27
Changed lines of the file:
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@@
+	)
+	(segment
+		(start 137.124341 87.34026)
+		(end 136.77521 87.689391)
+		(width 0.25)
+		(layer "F.Cu")
+		(net 1)
 	)
 	(segment
@@
 	)
 	(segment
+		(start 137.5511 87.34026)
+		(end 137.124341 87.34026)
+		(width 0.25)
+		(layer "F.Cu")
+		(net 1)
+	)
+	(segment
 		(start 143.797423 92.716583)
 		(end 143.4761 92.39526)
@@
 	)
 	(via
+		(at 136.77521 87.689391)
+		(size 0.8)
+		(drill 0.4)
+		(layers "F.Cu" "B.Cu")
+		(net 1)
+	)
+	(via
 		(at 130.9811 89.25026)
 		(size 0.8)
@@
 	)
 	(segment
+		(start 142.7961 87.69526)
+		(end 142.9961 87.89526)
+		(width 0.25)
+		(layer "F.Cu")
+		(net 2)
+	)
+	(segment
 		(start 131.8011 103.57026)
 		(end 138.3011 103.57026)
@@
 	)
 	(segment
+		(start 142.19856 87.69526)
+		(end 142.7961 87.69526)
+		(width 0.25)
+		(layer "F.Cu")
+		(net 2)
+	)
+	(segment
 		(start 128.541231 48.415195)
 		(end 128.541231 48.766641)
@@
 	)
 	(segment
-		(start 134.8261 91.32026)
-		(end 134.8261 90.54526)
-		(width 0.25)
-		(layer "F.Cu")
-		(net 2)
-	)
-	(segment
-		(start 134.8261 90.54526)
-		(end 135.0511 90.32026)
-		(width 0.25)
-		(layer "F.Cu")
-		(net 2)
-	)
-	(segment
 		(start 150.0611 77.82026)
 		(end 150.0611 77.037336)
@@
 	)
 	(segment
+		(start 136.0511 91.32026)
+		(end 134.8261 91.32026)
+		(width 0.25)
+		(layer "F.Cu")
+		(net 2)
+	)
+	(segment
 		(start 125.140038 79.56926)
 		(end 126.719212 79.56926)
@@
 	)
 	(segment
-		(start 140.9261 87.69526)
-		(end 142.7961 87.69526)
-		(width 0.25)
-		(layer "F.Cu")
-		(net 2)
-	)
-	(segment
 		(start 163.875401 78.170261)
 		(end 163.875401 79.32026)
@@
 	)
 	(segment
-		(start 142.7961 87.69526)
-		(end 142.9961 87.89526)
-		(width 0.25)
-		(layer "F.Cu")
-		(net 2)
-	)
-	(segment
 		(start 162.525399 88.120259)
 		(end 160.6754 86.27026)
@@
 	)
 	(via
-		(at 135.0511 90.32026)
+		(at 136.0511 91.32026)
 		(size 0.8)
 		(drill 0.4)
@@
 		(size 0.8)
 		(drill 0.4)
+		(layers "F.Cu" "B.Cu")
+		(net 2)
+	)
+	(via
+		(at 142.19856 87.69526)
+		(size 0.8)
+		(drill 0.4)
