File: MX_IMU.kicad_pcb (KiCad board)
At the start: 4 copper layers, 50 x 80 mm, 85 parts, among them J1 B2B-PH-K-S, J2 Native USB, J3 Native USB, J4 SM03B-GHS-TBLFSN, J5 Conn_02x03_Odd_Even, J6 Conn_02x03_Odd_Even, SW1 SSSS213000, SW2 SSSS213000, U1 CH340E, U10 ICM-42688-P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

Commit message: update
Parts:
- Reset1: footprint Button_Switch_THT:SW_PUSH_6mm -> Button_Switch_THT:SW_PUSH_6mm_H5mm
- U8: footprint Oscillator:Oscillator_SMD_SeikoEpson_SG8002CE-4Pin_3.2x2.5mm -> mylib:Oscillator_SMD_SeikoEpson_SG3225CAN-4Pin_3.2x2.5mm
- moved C20 0.44 mm to (139.6, 91.8), turned to 0 degrees
Routing:
- net +3.3V: track 68.5 -> 70.4 mm, vias 27 -> 29

Commit message: update
Parts:
- moved C26 3.50 mm to (156.1, 77.3), turned to 0 degrees
- moved C27 1.43 mm to (154.6, 81.3), turned to -90 degrees
- moved C25 0.60 mm to (155.5, 78.6)
Connections:
- net BARO_INT renamed Baro_INT
Routing:
- net Baro_INT: track 16.5 -> 15.6 mm
- net GND: track 169.5 -> 169.3 mm, vias 77 -> 79
Other:
- board text added: "IMU XO"
- board text removed: "32.768kXO"

Commit message: update
Parts:
- moved C24 2.69 mm to (150.6, 69.3)
- moved R12 2.24 mm to (148.1, 67.8), turned to -90 degrees
Routing:
- net Net-(U9-~{HOLD}/~{RESET}/IO_{3}): track 3.60 -> 2.47 mm
- net +3.3V: track 70.6 -> 69.7 mm, vias 29 -> 30
Changed lines of the file:
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@@
 	(footprint "Capacitor_SMD:C_0603_1608Metric"
 		(layer "F.Cu")
-		(at 148.0511 70.32026)
+		(at 150.5511 69.32026)
 		(descr "Capacitor SMD 0603 (1608 Metric), square (rectangular) end terminal, IPC-7351 nominal, (Body size source: IPC-SM-782 page 76, https://www.pcb-3d.com/wordpress/wp-content/uploads/ipc-sm-782a_amendment_1_and_2.pdf), generated with kicad-footprint-generator")
 		(tags "capacitor")
@@
 	(footprint "Resistor_SMD:R_0402_1005Metric"
 		(layer "F.Cu")
-		(at 150.0511 68.82026 180)
+		(at 148.0511 67.82026 -90)
 		(descr "Resistor SMD 0402 (1005 Metric), square (rectangular) end terminal, IPC-7351 nominal, (Body size source: IPC-SM-782 page 72, https://www.pcb-3d.com/wordpress/wp-content/uploads/ipc-sm-782a_amendment_1_and_2.pdf), generated with kicad-footprint-generator")
 		(tags "resistor")
 		(property "Reference" "R12"
-			(at -3 0 0)
+			(at -3 0 90)
 			(layer "F.SilkS")
 			(hide yes)
@@
 		)
 		(property "Value" "10k"
-			(at 0 1.17 0)
+			(at 0 1.17 90)
 			(layer "F.Fab")
 			(effects
@@
 		)
 		(property "Datasheet" "~"
-			(at 0 0 0)
+			(at 0 0 90)
 			(layer "F.Fab")
 			(hide yes)
@@
 		)
 		(property "Description" ""
-			(at 0 0 0)
+			(at 0 0 90)
 			(layer "F.Fab")
 			(hide yes)
@@
 		)
 		(property "LCSC Part #" "C25744"
-			(at 0 0 180)
+			(at 0 0 270)
 			(unlocked yes)
 			(layer "F.Fab")
@@
 		)
 		(fp_line
-			(start 0.93 0.47)
-			(end -0.93 0.47)
+			(start -0.93 0.47)
+			(end -0.93 -0.47)
 			(stroke
 				(width 0.05)
@@
 		)
 		(fp_line
-			(start 0.93 -0.47)
-			(end 0.93 0.47)
+			(start 0.93 0.47)
+			(end -0.93 0.47)
 			(stroke
 				(width 0.05)
@@
 		)
 		(fp_line
-			(start -0.93 0.47)
-			(end -0.93 -0.47)
+			(start -0.93 -0.47)
+			(end 0.93 -0.47)
 			(stroke
 				(width 0.05)
@@
 		)
 		(fp_line
-			(start -0.93 -0.47)
-			(end 0.93 -0.47)
+			(start 0.93 -0.47)
+			(end 0.93 0.47)
 			(stroke
 				(width 0.05)
@@
 		)
 		(fp_line
-			(start 0.525 0.27)
-			(end -0.525 0.27)
+			(start -0.525 0.27)
+			(end -0.525 -0.27)
 			(stroke
 				(width 0.1)
@@
 		)
 		(fp_line
-			(start 0.525 -0.27)
-			(end 0.525 0.27)
+			(start 0.525 0.27)
+			(end -0.525 0.27)
 			(stroke
 				(width 0.1)
@@
 		)
 		(fp_line
-			(start -0.525 0.27)
-			(end -0.525 -0.27)
+			(start -0.525 -0.27)
+			(end 0.525 -0.27)
 			(stroke
 				(width 0.1)
@@
 		)
 		(fp_line
-			(start -0.525 -0.27)
-			(end 0.525 -0.27)
+			(start 0.525 -0.27)
+			(end 0.525 0.27)
 			(stroke
 				(width 0.1)
@@
 		)
 		(fp_text user "${REFERENCE}"
-			(at 0 0 0)
+			(at 0 0 90)
 			(layer "F.Fab")
 			(effects
@@
 		)
 		(pad "1" smd roundrect
-			(at -0.51 0 180)
+			(at -0.51 0 270)
 			(size 0.54 0.64)
 			(layers "F.Cu" "F.Mask" "F.Paste")
@@
 		)
 		(pad "2" smd roundrect
-			(at 0.51 0 180)
+			(at 0.51 0 270)
 			(size 0.54 0.64)
 			(layers "F.Cu" "F.Mask" "F.Paste")
@@
 	)
 	(segment
+		(start 149.0511 69.32026)
+		(end 149.7761 69.32026)
+		(width 0.25)
+		(layer "F.Cu")
+		(net 1)
+	)
+	(segment
 		(start 155.0511 74.34026)
 		(end 155.0511 74.36026)
@@
 	)
 	(segment
+		(start 147.282404 69.088956)
+		(end 148.0411 68.33026)
+		(width 0.25)
+		(layer "F.Cu")
+		(net 1)
+	)
+	(segment
 		(start 146.0511 76.32026)
 		(end 146.4761 75.89526)
@@
 	)
 	(segment
+		(start 149.7761 67.41276)
+		(end 149.9636 67.22526)
+		(width 0.25)
+		(layer "F.Cu")
+		(net 1)
+	)
+	(segment
 		(start 155.008541 78.609783)
 		(end 155.008541 77.587819)
@@
 	)
 	(segment
-		(start 149.9636 66.95526)
-		(end 150.776099 66.95526)
-		(width 0.25)
-		(layer "F.Cu")
-		(net 1)
-	)
-	(segment
 		(start 132.3761 85.82026)
 		(end 132.3761 86.64526)
@@
 	)
 	(segment
-		(start 147.2761 70.09526)
-		(end 148.5511 68.82026)
-		(width 0.25)
-		(layer "F.Cu")
-		(net 1)
-	)
-	(segment
 		(start 155.276707 76.88835)
 		(end 155.276707 77.094653)
@@
 	)
 	(segment
+		(start 148.68125 69.690111)
+		(end 149.0511 69.32026)
+		(width 0.25)
+		(layer "F.Cu")
+		(net 1)
+	)
+	(segment
 		(start 139.0711 91.82026)
 		(end 139.0711 92.80026)
@@
 	)
 	(segment
-		(start 149.5411 67.64776)
-		(end 149.9636 67.22526)
-		(width 0.25)
-		(layer "F.Cu")
-		(net 1)
-	)
-	(segment
 		(start 155.480059 79.391301)
 		(end 155.480059 79.081301)
@@
 	)
 	(segment
-		(start 147.2761 70.32026)
-		(end 147.2761 70.09526)
-		(width 0.25)
-		(layer "F.Cu")
-		(net 1)
-	)
-	(segment
-		(start 149.5411 68.82026)
-		(end 148.5511 68.82026)
+		(start 149.5011 69.32026)
+		(end 149.5011 69.09526)
 		(width 0.25)
 		(layer "F.Cu")
@@
 	)
 	(segment
+		(start 149.7761 69.32026)
+		(end 149.7761 67.41276)
+		(width 0.25)
+		(layer "F.Cu")
+		(net 1)
+	)
+	(segment
 		(start 154.5511 80.84026)
 		(end 155.5311 80.84026)
@@
 	)
 	(segment
+		(start 148.0411 68.33026)
+		(end 148.0511 68.33026)
+		(width 0.25)
+		(layer "F.Cu")
+		(net 1)
+	)
+	(segment
 		(start 135.5511 86.59526)
 		(end 136.3261 85.82026)
@@
 	)
 	(segment
-		(start 149.5411 68.82026)
-		(end 149.5411 67.64776)
-		(width 0.25)
-		(layer "F.Cu")
-		(net 1)
-	)
-	(segment
 		(start 138.0511 73.97026)
 		(end 138.0511 75.32026)
@@
 	)
 	(via
-		(at 148.5511 68.82026)
+		(at 148.68125 69.690111)
 		(size 0.8)
 		(drill 0.4)
@@
 	)
 	(via
+		(at 147.282404 69.088956)
+		(size 0.8)
+		(drill 0.4)
+		(layers "F.Cu" "B.Cu")
+		(net 1)
+	)
+	(via
 		(at 139.0711 92.80026)
 		(size 0.8)
@@
 	)
 	(segment
-		(start 157.1386 63.41526)
-		(end 157.5511 63.00276)
-		(width 0.25)
-		(layer "F.Cu")
-		(net 2)
-	)
-	(segment
 		(start 151.079529 76.304857)
 		(end 151.294932 76.52026)
@@
 	)
 	(segment
-		(start 148.8261 70.32026)
-		(end 150.0511 70.32026)
-		(width 0.25)
-		(layer "F.Cu")
-		(net 2)
-	)
-	(segment
 		(start 147.704079 40.864515)
 		(end 147.105462 40.265898)
@@
 	)
 	(segment
-		(start 142.0886 63.70776)
-		(end 141.3011 63.70776)
+		(start 157.0511 62.32026)
+		(end 157.1386 62.40776)
 		(width 0.25)
 		(layer "F.Cu")
@@
 	)
 	(segment
-		(start 157.5511 63.00276)
-		(end 157.5511 62.32026)
+		(start 142.0886 63.70776)
+		(end 141.3011 63.70776)
 		(width 0.25)
 		(layer "F.Cu")
@@
 	)
 	(segment
+		(start 151.3261 69.32026)
+		(end 152.2761 69.32026)
+		(width 0.25)
+		(layer "F.Cu")
+		(net 2)
+	)
+	(segment
 		(start 140.9261 87.69526)
 		(end 140.9261 87.94526)
@@
 	)
 	(segment
+		(start 157.1386 62.40776)
+		(end 157.1386 63.41526)
+		(width 0.25)
+		(layer "F.Cu")
+		(net 2)
+	)
+	(segment
 		(start 152.634896 79.992591)
 		(end 152.634896 80.804083)
@@
 	)
 	(via
-		(at 157.5511 62.32026)
+		(at 157.0511 62.32026)
 		(size 0.8)
 		(drill 0.4)
@@
 	)
 	(via
-		(at 150.0511 70.32026)
+		(at 152.2761 69.32026)
 		(size 0.8)
 		(drill 0.4)
@@
 	)
 	(segment
-		(start 155.1461 67.22526)
-		(end 151.0511 71.32026)
+		(start 153.0511 70.82026)
+		(end 149.0511 70.82026)
 		(width 0.25)
 		(layer "F.Cu")
@@
 	)
 	(segment
-		(start 146.0511 73.47026)
-		(end 145.5511 73.97026)
+		(start 156.6461 67.22526)
+		(end 153.0511 70.82026)
 		(width 0.25)
 		(layer "F.Cu")
@@
 	)
 	(segment
-		(start 148.5511 71.32026)
+		(start 149.0511 70.82026)
 		(end 146.4011 73.47026)
 		(width 0.25)
@@
 	(segment
 		(start 157.1386 67.22526)
-		(end 155.1461 67.22526)
+		(end 156.6461 67.22526)
 		(width 0.25)
 		(layer "F.Cu")
@@
 	)
 	(segment
-		(start 151.0511 71.32026)
-		(end 148.5511 71.32026)
+		(start 146.0511 73.47026)
+		(end 145.5511 73.97026)
 		(width 0.25)
 		(layer "F.Cu")
@@
 	)
 	(segment
-		(start 157.1386 67.22526)
-		(end 158.9761 67.22526)
+		(start 146.4011 73.47026)
+		(end 146.0511 73.47026)
 		(width 0.25)
 		(layer "F.Cu")
@@
 	)
 	(segment
-		(start 146.4011 73.47026)
-		(end 146.0511 73.47026)
+		(start 157.1386 67.22526)
+		(end 158.9761 67.22526)
 		(width 0.25)
 		(layer "F.Cu")
@@
 	)
 	(segment
-		(start 150.776099 65.95526)
-		(end 151.5511 66.730261)
-		(width 0.25)
-		(layer "F.Cu")
-		(net 87)
-	)
-	(segment
-		(start 151.5511 66.730261)
-		(end 151.5511 67.83026)
+		(start 148.0511 67.31026)
+		(end 149.4061 65.95526)
 		(width 0.25)
 		(layer "F.Cu")
@@
 	)
 	(segment
-		(start 151.5511 67.83026)
-		(end 150.5611 68.82026)
+		(start 149.4061 65.95526)
+		(end 149.9636 65.95526)
 		(width 0.25)
 		(layer "F.Cu")

Commit message: update spi flash
Parts:
- U9: value W25Q128JVS -> W25Q128JVSIQ
Changed lines of the file:
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@@
 			)
 		)
-		(property "Datasheet" ""
+		(property "Datasheet" "https://www.lcsc.com/datasheet/C2650753.pdf"
 			(at 0 0 0)
 			(layer "F.Fab")
@@
 			)
 		)
-		(property "Description" ""
+		(property "Description" "3.3V 3.5mA CMOS SMD3225-4P Crystals RoHS 25ppm"
 			(at 0 0 0)
 			(layer "F.Fab")
@@
 			)
 		)
+		(property "LCSC Part " "C2650753"
+			(at 0 0 0)
+			(unlocked yes)
+			(layer "F.Fab")
+			(hide yes)
+			(effects
+				(font
+					(size 1 1)
+					(thickness 0.15)
+				)
+			)
+		)
 		(sheetname "/Peripherals/")
 		(sheetfile "Periph.kicad_sch")
@@
 			)
 		)
-		(property "Value" "W25Q128JVS"
+		(property "Value" "W25Q128JVSIQ"
 			(at 0 3.6 0)
 			(layer "F.Fab")
@@
 					(thickness 0.15)
 				)
+			)
+		)
+		(property "LCSC Part " "C97521"
+			(at 0 0 180)
+			(unlocked yes)
+			(layer "F.Fab")
+			(hide yes)
+			(effects
+				(font
+					(size 1 1)
+					(thickness 0.15)
+				)
