File: MX_IMU.kicad_pcb (KiCad board)
At the start: 4 copper layers, 50 x 80 mm, 85 parts, among them J1 B2B-PH-K-S, J2 Native USB, J3 Native USB, J4 SM03B-GHS-TBLFSN, J5 Conn_02x03_Odd_Even, J6 Conn_02x03_Odd_Even, SW1 SSSS213000, SW2 SSSS213000, U1 CH340E, U10 ICM-42688-P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

Commit message: update
Parts:
- moved C30 4.84 mm to (129.6, 75.8), turned to 0 degrees
- moved R14 0.50 mm to (132.1, 85.8)
- moved C28 0.34 mm to (129.6, 90.3), turned to 90 degrees
Routing:
- net +3.3V: track 69.7 -> 71.3 mm, vias 30 -> 31
- net GND: track 168.9 -> 170.3 mm, vias 79 -> 83
- net Baro_SCL: track 22.6 -> 21.6 mm
- net Baro_SDA: track 22.5 -> 21.5 mm
- net Baro_INT: track 15.6 -> 16.3 mm

Commit message: update
Parts:
- moved C29 2.83 mm to (130.6, 85.8), turned to 180 degrees
- moved R14 2.32 mm to (131.6, 88.1), turned to -90 degrees
- moved R15 1.10 mm to (128.6, 84.3)
- moved C28 1.09 mm to (129.0, 89.4), turned to 0 degrees
- moved U11 0.73 mm to (129.1, 87.6)
Routing:
- net Baro_SCL: track 21.6 -> 26.9 mm, vias 2 -> 3
- net +3.3V: track 71.3 -> 68.2 mm, vias 31 -> 32
- net Baro_INT: track 16.3 -> 17.9 mm
- net Baro_SDA: track 21.5 -> 22.4 mm, vias 2 -> 0
- net +5V: track 123.3 -> 122.7 mm
- net GND: track 170.3 -> 170.1 mm, vias 83 -> 81

Commit message: update
Parts:
- moved J1 1.34 mm to (120.6, 41.3)
- moved SW2 1.00 mm to (150.1, 100.3)
- moved Reset1 0.50 mm to (131.8, 98.6)
Routing:
- net VCC: track 11.7 -> 10.2 mm
- net +5V: track 122.7 -> 121.6 mm
- net BOOT0: track 27.3 -> 26.3 mm
- net GND: track 170.1 -> 170.7 mm
Changed lines of the file:
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@@
 	(footprint "Button_Switch_THT:SW_PUSH_6mm_H5mm"
 		(layer "F.Cu")
-		(at 131.8011 99.07026)
+		(at 131.8011 98.57026)
 		(descr "tactile push button, 6x6mm e.g. PHAP33xx series, height=5mm")
 		(tags "tact sw push 6mm")
@@
 	(footprint "mylib:SSSS213000"
 		(layer "F.Cu")
-		(at 150.0511 101.32026 180)
+		(at 150.0511 100.32026 180)
 		(descr "SSSS213000")
 		(tags "Schottky Diode")
@@
 	(footprint "mylib:JST_B2B-PH-K-S"
 		(layer "F.Cu")
-		(at 119.3011 41.64526 -90)
+		(at 120.6011 41.32026 -90)
 		(property "Reference" "J1"
 			(at 3.725 -3.63 90)
@@
 	)
 	(gr_text "VCC\n"
-		(at 122.198301 42.9508 0)
+		(at 124.0511 42.783857 0)
 		(layer "F.SilkS")
 		(effects
@@
 	)
 	(gr_text "GND"
-		(at 154.0511 105.32026 0)
+		(at 154.0511 104.32026 0)
 		(layer "F.SilkS")
 		(effects
@@
 	)
 	(gr_text "GND\n"
-		(at 122.173714 40.811687 0)
+		(at 124.0511 40.701887 0)
 		(layer "F.SilkS")
 		(effects
@@
 	)
 	(gr_text "3.3V\n"
-		(at 145.0511 105.32026 0)
+		(at 145.0511 104.32026 0)
 		(layer "F.SilkS")
 		(effects
@@
 	)
 	(segment
-		(start 147.5511 102.97026)
-		(end 144.7011 102.97026)
+		(start 147.5511 101.97026)
+		(end 144.7011 101.97026)
 		(width 0.25)
 		(layer "F.Cu")
@@
 	)
 	(via
-		(at 144.7011 102.97026)
+		(at 144.7011 101.97026)
 		(size 0.8)
 		(drill 0.4)
@@
 	)
 	(segment
-		(start 118.7511 40.64526)
-		(end 120.0511 40.64526)
-		(width 0.5)
-		(layer "F.Cu")
-		(net 2)
-	)
-	(segment
 		(start 129.0511 88.35026)
 		(end 128.5511 88.35026)
@@
 	)
 	(via
-		(at 120.0511 40.64526)
-		(size 0.8)
-		(drill 0.4)
-		(layers "F.Cu" "B.Cu")
-		(net 2)
-	)
-	(via
 		(at 146.8011 34.57026)
 		(size 0.8)
@@
 	)
 	(via
+		(at 121.5511 39.32026)
+		(size 0.8)
+		(drill 0.4)
+		(layers "F.Cu" "B.Cu")
+		(net 2)
+	)
+	(via
 		(at 156.903573 78.579912)
 		(size 0.8)
@@
 	)
 	(segment
+		(start 120.0511 40.32026)
+		(end 121.0511 39.32026)
+		(width 0.25)
+		(layer "B.Cu")
+		(net 2)
+	)
+	(segment
+		(start 121.0511 39.32026)
+		(end 121.5511 39.32026)
+		(width 0.25)
+		(layer "B.Cu")
+		(net 2)
+	)
+	(segment
 		(start 138.614563 45.683723)
 		(end 138.5761 45.64526)
@@
 	)
 	(segment
-		(start 156.9761 52.32026)
-		(end 163.8011 59.14526)
+		(start 140.235262 52.32026)
+		(end 156.9761 52.32026)
 		(width 0.8)
 		(layer "In2.Cu")
@@
 	)
 	(segment
+		(start 161.0511 75.64526)
+		(end 161.0511 78.39526)
+		(width 0.8)
+		(layer "In2.Cu")
+		(net 3)
+	)
+	(segment
 		(start 131.3311 55.04026)
 		(end 124.0511 62.32026)
@@
 	)
 	(segment
-		(start 163.8011 72.89526)
-		(end 161.0511 75.64526)
-		(width 0.8)
+		(start 120.5511 76.82026)
+		(end 124.0511 73.32026)
+		(width 0.5)
 		(layer "In2.Cu")
 		(net 3)
 	)
 	(segment
-		(start 163.8011 59.14526)
-		(end 163.8011 72.89526)
-		(width 0.8)
+		(start 121.698851 66.043011)
+		(end 124.0511 68.39526)
+		(width 0.5)
 		(layer "In2.Cu")
 		(net 3)
@@
 	)
 	(segment
-		(start 138.718181 53.837341)
-		(end 140.235262 52.32026)
+		(start 128.0511 75.82026)
+		(end 126.5511 75.82026)
 		(width 0.8)
 		(layer "In2.Cu")
@@
 	)
 	(segment
-		(start 161.0511 75.64526)
-		(end 161.0511 78.39526)
+		(start 162.5511 57.89526)
+		(end 162.5511 74.14526)
 		(width 0.8)
 		(layer "In2.Cu")
@@
 	)
 	(segment
-		(start 120.5511 76.82026)
+		(start 124.0511 68.39526)
 		(end 124.0511 73.32026)
-		(width 0.5)
-		(layer "In2.Cu")
-		(net 3)
-	)
-	(segment
-		(start 121.698851 66.043011)
-		(end 124.0511 68.39526)
-		(width 0.5)
+		(width 0.8)
 		(layer "In2.Cu")
 		(net 3)
 	)
 	(segment
-		(start 128.0511 75.82026)
-		(end 126.5511 75.82026)
+		(start 135.7261 55.04026)
+		(end 131.3311 55.04026)
 		(width 0.8)
 		(layer "In2.Cu")
@@
 	)
 	(segment
-		(start 124.0511 68.39526)
-		(end 124.0511 73.32026)
+		(start 162.5511 74.14526)
+		(end 161.0511 75.64526)
 		(width 0.8)
 		(layer "In2.Cu")
@@
 	)
 	(segment
-		(start 135.7261 55.04026)
-		(end 131.3311 55.04026)
+		(start 156.9761 52.32026)
+		(end 162.5511 57.89526)
 		(width 0.8)
 		(layer "In2.Cu")
@@
 	)
 	(segment
-		(start 140.235262 52.32026)
-		(end 156.9761 52.32026)
+		(start 138.718181 53.837341)
+		(end 140.235262 52.32026)
 		(width 0.8)
 		(layer "In2.Cu")
@@
 	)
 	(segment
-		(start 118.8011 46.37026)
-		(end 121.7511 49.32026)
-		(width 2)
-		(layer "F.Cu")
-		(net 6)
-	)
-	(segment
-		(start 119.43235 45.73901)
-		(end 118.8011 46.37026)
+		(start 121.2511 46.32026)
+		(end 120.0511 45.12026)
 		(width 1)
 		(layer "F.Cu")
@@
 	)
 	(segment
-		(start 118.7511 42.64526)
-		(end 118.8011 42.69526)
+		(start 120.0511 47.62026)
+		(end 121.7511 49.32026)
 		(width 2)
 		(layer "F.Cu")
@@
 	)
 	(segment
-		(start 118.8011 42.69526)
-		(end 118.8011 46.37026)
+		(start 120.0511 42.32026)
+		(end 120.0511 45.12026)
 		(width 2)
 		(layer "F.Cu")
@@
 	)
 	(segment
-		(start 121.46985 45.73901)
-		(end 119.43235 45.73901)
-		(width 1)
+		(start 120.0511 45.12026)
+		(end 120.0511 47.62026)
+		(width 2)
 		(layer "F.Cu")
 		(net 6)
@@
 	(segment
 		(start 122.0511 46.32026)
-		(end 121.46985 45.73901)
+		(end 121.2511 46.32026)
 		(width 1)
 		(layer "F.Cu")
@@
 	(segment
 		(start 147.0511 88.49526)
-		(end 146.0511 88.49526)
+		(end 150.0511 91.49526)
 		(width 0.25)
 		(layer "F.Cu")
@@
 	)
 	(segment
-		(start 150.0511 91.49526)
-		(end 150.0511 99.67026)
+		(start 147.0511 88.49526)
+		(end 146.0511 88.49526)
 		(width 0.25)
 		(layer "F.Cu")
@@
 	)
 	(segment
-		(start 147.0511 88.49526)
-		(end 150.0511 91.49526)
+		(start 150.0511 91.49526)
+		(end 150.0511 98.67026)
 		(width 0.25)
 		(layer "F.Cu")
@@
 		(polygon
 			(pts
-				(xy 167.3011 25.64526) (xy 167.3011 108.14526) (xy 114.8011 108.14526) (xy 114.8011 25.64526)
+				(xy 163.8011 29.64526) (xy 163.8011 104.14526) (xy 117.8011 104.14526) (xy 117.8011 29.64526)
 			)
 		)

Commit message: update
Parts:
- moved C28 3.66 mm to (127.0, 86.3), turned to -90 degrees
- moved R14 3.35 mm to (128.3, 88.8), turned to 180 degrees
- moved C30 3.02 mm to (126.5, 75.8), turned to 180 degrees
- moved R15 2.69 mm to (131.1, 85.3), turned to 90 degrees
- moved C29 1.55 mm to (131.1, 87.3)
- moved U11 1.29 mm to (128.8, 86.3), turned to 90 degrees
Routing:
- net Baro_INT: track 17.9 -> 10.2 mm, vias 2 -> 0
- net Baro_SCL: track 26.9 -> 24.5 mm
- net SWO: track 11.9 -> 13.6 mm
- net Baro_SDA: track 22.4 -> 20.8 mm, vias 0 -> 2
- net +3.3V: track 68.2 -> 69.4 mm, vias 32 -> 31
- net GND: track 170.7 -> 172.0 mm
- net GPS_TX: track 19.6 -> 20.6 mm, vias 0 -> 2
- net +5V: track 121.6 -> 121.1 mm
- net GPS_RX: track 19.3 -> 19.7 mm, vias 0 -> 2
